File: LCD_Adapter/LCD_Adapter/LCD_Adapter.kicad_sch (KiCad schematic)
At the start: 29 parts, among them J1 Conn_01x10, J2 FH12-30S-0.5SH_55_, J3 Conn_01x22, U1 TLV75801PDBV, U2 TLV75801PDBV, U3 TPS61042DRBR

Commit message: PCD_UPDATE
Parts:
- removed C1, C3, C4, C5: 0.47uF, Capacitor_SMD:C_0603_1608Metric, symbol Device:C
- removed C2, C6, C8: 4.7uF, Capacitor_SMD:C_0603_1608Metric, symbol Device:C
- removed C7: 1uF, Capacitor_SMD:C_0603_1608Metric, symbol Device:C
- removed D1: 1N5819WS, Diode_SMD:D_SOD-323, symbol Diode:1N5819WS
- removed J1: Conn_01x10, Connector_PinHeader_2.54mm:PinHeader_1x10_P2.54mm_Vertical, symbol Connector_Generic:Conn_01x10
- removed J2: FH12-30S-0.5SH_55_, lib:HIROSE_FH12-30S-0.5SH_55_, symbol FH12-30S-0.5SH_55_:FH12-30S-0.5SH_55_
- removed J3: Conn_01x22, lib:FC-10A20P11H20, symbol Connector_Generic:Conn_01x22
- removed L1: L, Inductor_SMD:L_1210_3225Metric, symbol Device:L
- removed R1, R2, R3, R4, R5: 0, Resistor_SMD:R_0603_1608Metric, symbol Device:R
- removed R12: 39k, Resistor_SMD:R_0603_1608Metric, symbol Device:R
- removed R13: 160k, Resistor_SMD:R_0603_1608Metric, symbol Device:R
- removed R14: 230k, Resistor_SMD:R_0603_1608Metric, symbol Device:R
- removed R15: 100k, Resistor_SMD:R_0603_1608Metric, symbol Device:R
- removed R16: 6.8, Resistor_SMD:R_0603_1608Metric, symbol Device:R
- removed TP2, TP3, TP4: TestPoint, TestPoint:TestPoint_Pad_D1.0mm, symbol Connector:TestPoint
- removed U1, U2: TLV75801PDBV, Package_TO_SOT_SMD:SOT-23-5, symbol Regulator_Linear:TLV75801PDBV
- removed U3: TPS61042DRBR, lib:DRB8_1P75X1P5, symbol TPS61042:TPS61042DRBR
Other:
- added sheet PWR (PWM.kicad_sch)
- added sheet RPI2LCD (RPI2LCD.kicad_sch)
- added sheet STM2LCD (STM2LCD.kicad_sch)
