File: PCB/DAC.kicad_sch (KiCad schematic)
At the start: 1 part, among them J1 SJ3-35024K-SMT-TR

Commit message: PCB_UPDATE
Parts:
- removed J1: SJ3-35024K-SMT-TR, SJ3-35024K-SMT-TR:SAMESKY_SJ3-35024K-SMT-TR, symbol SJ3-35024K-SMT-TR:SJ3-35024K-SMT-TR
- added J1: SJ-43504-SMT-TR, lib:CUI_SJ-43504-SMT-TR, symbol SJ-43504-SMT-TR:SJ-43504-SMT-TR
Changed lines of the file:
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@@
 	)
 	(symbol
-		(lib_id "SJ3-35024K-SMT-TR:SJ3-35024K-SMT-TR")
-		(at 125.73 64.77 0)
+		(lib_id "SJ-43504-SMT-TR:SJ-43504-SMT-TR")
+		(at 78.74 66.04 0)
 		(unit 1)
 		(exclude_from_sim no)
@@
 		(fields_autoplaced yes)
 		(property "Reference" "J1"
-			(at 125.095 49.53 0)
+			(at 74.6125 55.88 0)
 			(effects
 				(font
@@
 			)
 		)
-		(property "Value" "SJ3-35024K-SMT-TR"
-			(at 125.095 52.07 0)
+		(property "Value" "SJ-43504-SMT-TR"
+			(at 74.6125 58.42 0)
 			(effects
 				(font
@@
 			)
 		)
-		(property "Footprint" "SJ3-35024K-SMT-TR:SAMESKY_SJ3-35024K-SMT-TR"
-			(at 125.73 64.77 0)
+		(property "Footprint" "lib:CUI_SJ-43504-SMT-TR"
+			(at 78.74 66.04 0)
 			(effects
 				(font
@@
 		)
 		(property "Datasheet" ""
-			(at 125.73 64.77 0)
+			(at 78.74 66.04 0)
 			(effects
 				(font
@@
 		)
 		(property "Description" ""
-			(at 125.73 64.77 0)
+			(at 78.74 66.04 0)
 			(effects
 				(font
@@
 			)
 		)
-		(property "PARTREV" "1.0"
-			(at 125.73 64.77 0)
+		(property "MF" "Same Sky"
+			(at 78.74 66.04 0)
+			(effects
+				(font
+					(size 1.27 1.27)
+				)
+				(justify bottom)
+				(hide yes)
+			)
+		)
+		(property "MAXIMUM_PACKAGE_HEIGHT" "3.3 mm"
+			(at 78.74 66.04 0)
+			(effects
+				(font
+					(size 1.27 1.27)
+				)
+				(justify bottom)
+				(hide yes)
+			)
+		)
+		(property "Package" "None"
+			(at 78.74 66.04 0)
+			(effects
+				(font
+					(size 1.27 1.27)
+				)
+				(justify bottom)
+				(hide yes)
+			)
+		)
+		(property "Price" "None"
+			(at 78.74 66.04 0)
+			(effects
+				(font
+					(size 1.27 1.27)
+				)
+				(justify bottom)
+				(hide yes)
+			)
+		)
+		(property "Check_prices" "https://www.snapeda.com/parts/SJ-43504-SMT-TR/Same+Sky/view-part/?ref=eda"
+			(at 78.74 66.04 0)
 			(effects
 				(font
@@
 		)
 		(property "STANDARD" "Manufacturer Recommendations"
-			(at 125.73 64.77 0)
+			(at 78.74 66.04 0)
 			(effects
 				(font
@@
 			)
 		)
-		(property "MAXIMUM_PACKAGE_HEIGHT" "5.575mm"
-			(at 125.73 64.77 0)
+		(property "PARTREV" "10/08/2019"
+			(at 78.74 66.04 0)
 			(effects
 				(font
@@
 			)
 		)
-		(property "MANUFACTURER" "Same Sky"
-			(at 125.73 64.77 0)
+		(property "SnapEDA_Link" "https://www.snapeda.com/parts/SJ-43504-SMT-TR/Same+Sky/view-part/?ref=snap"
+			(at 78.74 66.04 0)
 			(effects
 				(font
@@
 			)
 		)
-		(pin "8"
+		(property "MP" "SJ-43504-SMT-TR"
+			(at 78.74 66.04 0)
+			(effects
+				(font
+					(size 1.27 1.27)
+				)
+				(justify bottom)
+				(hide yes)
+			)
+		)
+		(property "Description_1" "3.5 mm, Stereo, Right Angle, Mid Mount (SMT), Shielded, 4 Conductors, 2 Internal Switches, Audio Jack Connector"
+			(at 78.74 66.04 0)
+			(effects
+				(font
+					(size 1.27 1.27)
+				)
+				(justify bottom)
+				(hide yes)
+			)
+		)
+		(property "MANUFACTURER" "CUI Devices"
+			(at 78.74 66.04 0)
+			(effects
+				(font
+					(size 1.27 1.27)
+				)
+				(justify bottom)
+				(hide yes)
+			)
+		)
+		(property "Availability" "In Stock"
+			(at 78.74 66.04 0)
+			(effects
+				(font
+					(size 1.27 1.27)
+				)
+				(justify bottom)
+				(hide yes)
+			)
+		)
+		(property "SNAPEDA_PN" "SJ-43504-SMT-TR"
+			(at 78.74 66.04 0)
+			(effects
+				(font
+					(size 1.27 1.27)
+				)
+				(justify bottom)
+				(hide yes)
+			)
+		)
+		(pin "6"
 		)
 		(pin "2"
@@
 		(pin "4"
 		)
-		(pin "7"
+		(pin "1"
 		)
 		(pin "3"
 		)
-		(pin "1"
-		)
-		(pin "6"
-		)
 		(instances
