File: PCB/MPU_MOD.kicad_pcb (KiCad board)
At the start: 8 copper layers, 43.5 x 70 mm, 305 parts, among them J1 SJ-43504-SMT-TR, J2 2-1734248-0, J3 USB4510-03-1-A_REVA, J501 MEM2090-00-145-00-A_REVA, J701 FTSH-107-01-L-DV-K-A, J901 73412-0110, U1 IS21ES08GA-JQLI-TR, U201 STC3115IQT, U203 STPMIC1APQR, U3 BQ24298RTWR, U301 STM32MP157FABx, U401 MT41K256M16TW-107_P, U502 HSP051-4M10, U503 HSP051-4M10, U701 HSP051-4M10, U702 HSP051-4M10, U801 FUSB302BMPX, U802 HSP051-4M10, U901 LBEE5PK2AE-771, Y601 NX2012SA-32.768K, Y701 ECS-2520MVQ-240

Commit message: PCB_UPDATE
Parts:
- removed TP201, TP202, TP204, TP205, TP206, TP207, TP208, TP209, TP210, TP211, TP212, TP401, TP402, TP403, TP601, TP602, TP701, TP702, TP703, TP704, TP705, TP706, TP707, TP708, TP709, TP710, TP801, TP803, TP804, TP805, TP806, TP901, TP902, TP903, TP904, TP905, TP906, TP907, TP908: TestPoint, Library:TP_0.5mm
- moved S702 123.4 mm to (40.7, 43.6)
- moved R706 115.9 mm to (35.7, 59.6)
- moved R709 115.9 mm to (38.6, 53.6)
- moved R710 115.9 mm to (38.6, 55.6)
- moved R715 100.1 mm to (38.6, 57.6)
- moved J701 98.4 mm to (45.8, 52.9)
- moved U701 88.5 mm to (53.6, 50.1)
- moved U702 88.5 mm to (53.6, 53.1)
- moved C803 75.9 mm to (46.8, 63.6), turned to 0 degrees
- moved C804 73.9 mm to (46.8, 65.6), turned to 0 degrees
- moved C805 71.2 mm to (50.2, 63.9), turned to 0 degrees
- moved R603 63.6 mm to (59.0, 53.4)
- moved S701 63.2 mm to (50.8, 40.7), turned to 0 degrees
- moved R604 63.2 mm to (59.0, 55.4)
- moved R701 61.8 mm to (35.7, 49.7)
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Connections:
- U401 pad E3: /DDR/DDR_DQ9 -> /DDR/DDR_DQ13
- U401 pad H3: /DDR/DDR_DQ13 -> /DDR/DDR_DQ9
Routing:
- net GND: track 88.9 -> 98.3 mm, vias 102 -> 106
- net /DDR/DDR_DQ11: track 17.1 -> 24.9 mm
- net VDD_DDR: track 33.5 -> 41.1 mm, vias 25 -> 27
- net /DDR/DDR_DQ13: track 18.4 -> 25.9 mm
- net /DDR/DDR_DQS1_N: track 18.1 -> 25.5 mm
- net /DDR/DDR_DQS1_P: track 19.0 -> 25.7 mm
- net /DDR/DDR_DQM1: track 20.5 -> 26.1 mm
- net /DDR/DDR_DQ14: track 20.7 -> 25.6 mm
- net /DDR/DDR_RESETN: track 13.3 -> 17.8 mm, vias 1 -> 2
- net /DDR/DDR_DQ9: track 22.0 -> 25.4 mm
- net /DDR/DDR_DQ15: track 22.5 -> 25.1 mm
- net VREF_DDR: track 7.25 -> 9.56 mm, vias 2 -> 3
- net /DDR/DDR_DQ8: track 25.3 -> 27.3 mm
- net /DDR/DDR_DQ10: track 24.3 -> 26.0 mm
- net /DDR/DDR_CSN: track 29.7 -> 31.0 mm
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
Commit message: PCB_update
Connections:
- U401 pad A2: /DDR/DDR_DQ0 -> /DDR/DDR_DQ3
- U401 pad B8: /DDR/DDR_DQ5 -> /DDR/DDR_DQ4
- U401 pad C2: /DDR/DDR_DQ3 -> /DDR/DDR_DQ0
- U401 pad C8: /DDR/DDR_DQ4 -> /DDR/DDR_DQ5
Routing:
- net /DDR/DDR_DQM0: track 22.4 -> 25.1 mm
- net /DDR/DDR_DQ1: track 22.2 -> 23.8 mm
- net /DDR/DDR_DQ5: track 25.2 -> 24.1 mm
- net /DDR/DDR_DQ0: track 25.3 -> 24.2 mm
- net /DDR/DDR_DQ7: track 23.7 -> 24.6 mm
- net /DDR/DDR_DQ3: track 24.4 -> 25.3 mm
- net /DDR/DDR_A0: track 29.4 -> 28.7 mm
