File: PCB/MPU_MOD.kicad_pcb (KiCad board)
At the start: 6 copper layers, 43.5 x 90 mm, 292 parts, among them J1 SJ-43504-SMT-TR, J2 2-1734248-0, J3 USB4510-03-1-A_REVA, J501 MEM2090-00-145-00-A_REVA, J701 FTSH-107-01-L-DV-K-A, J901 73412-0110, U201 STC3115IQT, U203 STPMIC1APQR, U3 BQ24298RTWR, U301 STM32MP157FABx, U401 MT41K256M16TW-107_P, U502 HSP051-4M10, U503 HSP051-4M10, U701 HSP051-4M10, U702 HSP051-4M10, U801 FUSB302BMPX, U802 HSP051-4M10, U901 LBEE5PK2AE-771, Y601 NX2012SA-32.768K, Y701 ECS-2520MVQ-240

Commit message: PCB_UPDATE
Parts:
- added J4: Conn_02x20_Odd_Even, Connector_PinHeader_1.27mm:PinHeader_2x20_P1.27mm_Horizontal, F.Cu at (77.7, 43.4)
- moved S602 39.0 mm to (71.4, 62.4)
- moved J901 27.9 mm to (71.5, 90.0)
- moved C904 26.4 mm to (81.0, 101.5)
- moved C903 26.0 mm to (73.0, 104.0)
- moved C905 26.0 mm to (79.5, 103.7)
- moved L901 26.0 mm to (76.7, 103.3)
- moved R902 26.0 mm to (77.7, 94.0)
- moved U901 26.0 mm to (73.1, 98.0)
- moved C901 26.0 mm to (80.9, 104.1)
- moved C902 26.0 mm to (78.9, 101.3)
- moved R901 26.0 mm to (78.7, 94.0)
- moved R903 25.7 mm to (72.5, 92.8)
- moved J501 18.6 mm to (68.5, 77.4)
- moved NT1 18.6 mm to (70.8, 83.4)
- moved R513 18.6 mm to (79.8, 82.5)
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Connections:
- net SDMMC2_D0 renamed I2S2_SDI
- net SDMMC2_D1 renamed I2S2_SDO
- net SDMMC2_D2 renamed I2S3_CK
- net SDMMC2_D3 renamed I2S3_SDI
- net SDMMC2_D4 renamed I2S3_SDO
- net SDMMC2_D5 renamed I2S2_CK
- U301 pad A5: SDMMC2_CK -> unconnected-(U301D-PE3-PadA5)
- U301 pad A6: SDMMC2_CMD -> unconnected-(U301D-PG6-PadA6)
- U301 pad B7: SDMMC2_D6 -> unconnected-(U301D-PE5-PadB7)
- U301 pad C6: SDMMC2_D7 -> unconnected-(U301C-PD3-PadC6)
- U301 pad C7: unconnected-(U301C-PA15-PadC7) -> I2S3_WS
- U301 pad D9: unconnected-(U301C-PB9-PadD9) -> I2S2_WS
- U301 pad P4: I2S1_CK -> unconnected-(U301C-PA5-PadP4)
- U301 pad R4: I2S1_WS -> unconnected-(U301C-PA4-PadR4)
- U301 pad T2: I2S1_SDI -> unconnected-(U301C-PC2-PadT2)
- U301 pad T5: I2S1_SDI -> unconnected-(U301C-PA6-PadT5)
- U301 pad T6: I2S1_SDO -> unconnected-(U301C-PA7-PadT6)
- U301 pad V2: I2S1_SDO -> unconnected-(U301C-PC1-PadV2)
- U301 pad V5: I2S1_WS -> unconnected-(U301C-PB12-PadV5)
- U301 pad W5: I2S1_CK -> unconnected-(U301C-PB10-PadW5)
Routing:
- net DSI_D2_P: track 4.31 -> 55.9 mm
- net DSI_CK_P: track 4.44 -> 30.6 mm
- net DSI_CK_N: track 3.27 -> 29.0 mm
- net DSI_D1_N: track 3.40 -> 27.0 mm
- net SDMMC1_D0: track 17.9 -> 31.8 mm
- net SDMMC1_D2: track 15.7 -> 29.3 mm
- net I2S3_WS: track 0.00 -> 13.5 mm
- net I2S2_WS: track 0.00 -> 12.9 mm, vias 0 -> 1
- net SDMMC1_D3: track 11.5 -> 23.9 mm
- net I2S2_CK: track 0.02 -> 11.4 mm, vias 0 -> 1
- net I2S2_SDI: track 0.02 -> 11.3 mm, vias 0 -> 1
- net SDMMC3_D2: track 0.00 -> 11.2 mm, vias 0 -> 1
- net I2S3_SDO: track 0.00 -> 10.7 mm
- net I2S3_CK: track 0.00 -> 10.6 mm
- net I2S2_SDO: track 0.00 -> 9.50 mm, vias 0 -> 1
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
Commit message: PCB_UPDATE
Connections:
- U301 pad T10: unconnected-(U301D-PE7-PadT10) -> UART7_RX_STM
- U301 pad T11: unconnected-(U301D-PE8-PadT11) -> UART7_TX_STM
- U301 pad T12: unconnected-(U301C-PB6-PadT12) -> FDCAN2_TX
- U301 pad U16: unconnected-(U301C-PA12-PadU16) -> SYS_I2C6_SDA
- U301 pad V14: unconnected-(U301F-USB_DP1-PadV14) -> USB_M_D+
- U301 pad V17: unconnected-(U301C-PA11-PadV17) -> SYS_I2C6_SCL
- U301 pad V5: unconnected-(U301C-PB12-PadV5) -> FDCAN2_RX
- U301 pad W14: unconnected-(U301F-USB_DM1-PadW14) -> USB_M_D-
Routing:
- net USB_M_D+: track 0.00 -> 31.5 mm
- net USB_M_D-: track 0.00 -> 30.0 mm
- net FDCAN2_RX: track 0.00 -> 16.9 mm, vias 0 -> 2
- net FDCAN2_TX: track 0.00 -> 12.1 mm, vias 0 -> 2
- net UART7_RX_STM: track 0.00 -> 10.8 mm, vias 0 -> 2
- net UART7_TX_STM: track 0.00 -> 10.7 mm, vias 0 -> 2
- net SYS_I2C6_SDA: track 0.00 -> 8.97 mm, vias 0 -> 2
- net SYS_I2C6_SCL: track 0.00 -> 8.04 mm, vias 0 -> 2
- net SYS_I2C4_SCL: track 41.3 -> 43.8 mm
- net GND: track 191.8 -> 192.2 mm, vias 186 -> 187

Commit message: psb_update
Parts:
- R715, U701, U702: moved to B.Cu
- TP703, TP704, TP705, TP706, TP707, TP708, TP709, TP710: moved to F.Cu
- moved TP705 48.5 mm to (61.1, 95.4), turned to 0 degrees
- moved TP704 48.0 mm to (59.6, 96.9), turned to 0 degrees
- moved TP703 47.4 mm to (59.6, 95.4), turned to 0 degrees
- moved TP709 45.3 mm to (64.1, 95.4), turned to 0 degrees
- moved TP710 44.8 mm to (64.1, 96.9), turned to 0 degrees
- moved TP708 44.8 mm to (62.6, 96.9), turned to 0 degrees
- moved TP707 43.9 mm to (62.6, 95.4), turned to 0 degrees
- moved TP706 43.4 mm to (61.1, 96.9), turned to 0 degrees
- moved R715 10.6 mm to (105.2, 108.6), turned to -90 degrees
- moved U702 9.49 mm to (102.2, 108.5), turned to 180 degrees
- moved U701 8.08 mm to (102.8, 121.4), turned to 180 degrees
- moved J701 1.65 mm to (102.7, 113.4), turned to 0 degrees
Connections:
- U301 pad T6: unconnected-(U301C-PA7-PadT6) -> ETH1_CRS_DV
- U301 pad T9: unconnected-(U301C-PB13-PadT9) -> ETH1_TXD1
- U301 pad U10: unconnected-(U301D-PF8-PadU10) -> SPI5_MISO
- U301 pad U2: unconnected-(U301D-PG13-PadU2) -> ETH1_TXD0
- U301 pad U4: PWR_SW_WAKE_UP -> ETH1_REF_CLK
- U301 pad V1: unconnected-(U301C-PB11-PadV1) -> ETH1_TX_EN
- U301 pad V2: unconnected-(U301C-PC1-PadV2) -> ETH1_MDC
- U301 pad V4: unconnected-(U301C-PC5-PadV4) -> ETH1_RXD1
- U301 pad W2: unconnected-(U301C-PA2-PadW2) -> ETH1_MDIO
- U301 pad W4: unconnected-(U301C-PC4-PadW4) -> ETH1_RXD0
- U301 pad W8: unconnected-(U301D-PF7-PadW8) -> SPI5_SCK
- U301 pad W9: unconnected-(U301D-PF9-PadW9) -> SPI5_MOSI
Routing:
- net UART4_RX_STM: track 0.58 -> 19.8 mm, vias 1 -> 2
- net ETH1_TX_EN: track 0.00 -> 13.4 mm, vias 0 -> 2
- net UART4_TX_STM: track 0.53 -> 9.75 mm, vias 1 -> 0
- net /RCC_BOOT_RST_DEBUG/T_JCLK/T_SWCLK: track 0.55 -> 9.53 mm
- net /RCC_BOOT_RST_DEBUG/T_JTMS/T_SWDIO: track 0.53 -> 9.31 mm
- net ETH1_TXD1: track 0.00 -> 8.58 mm, vias 0 -> 1
- net /RCC_BOOT_RST_DEBUG/T_JTDO/T_SWO: track 0.46 -> 8.97 mm
- net ETH1_TXD0: track 0.00 -> 8.40 mm, vias 0 -> 2
- net ETH1_CRS_DV: track 0.00 -> 8.40 mm, vias 0 -> 1
- net /RCC_BOOT_RST_DEBUG/T_JTDI/NC: track 0.60 -> 8.89 mm
- net ETH1_REF_CLK: track 0.00 -> 8.25 mm, vias 0 -> 1
- net ETH1_RXD1: track 0.00 -> 7.27 mm, vias 0 -> 1
- net ETH1_MDC: track 0.00 -> 7.18 mm, vias 0 -> 1
- net ETH1_RXD0: track 0.00 -> 5.94 mm, vias 0 -> 1
- net ETH1_MDIO: track 0.00 -> 5.65 mm, vias 0 -> 2
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