File: PCB/DDR.kicad_sch (KiCad schematic)
At the start: 65 parts, among them U301 STM32MP157FABx, U401 MT41K256M16TW-107_P

Commit message: PCB_UPDATE
Parts:
- renumbered C422 to C100, C423 to C101, C424 to C102, C425 to C103, C426 to C104, C427 to C105, C428 to C106, C429 to C107, C430 to C108, C401 to C79, C402 to C80, C403 to C81, C404 to C82, C405 to C83, C406 to C84, C407 to C85, C408 to C86, C409 to C87, C410 to C88, C411 to C89, C412 to C90, C413 to C91, C414 to C92, C415 to C93, C416 to C94, C417 to C95, C418 to C96, C419 to C97, C420 to C98, C421 to C99, R401 to R17, R402 to R18, R403 to R19, R404 to R20, R405 to R21, R406 to R22, R407 to R23, R408 to R24, R409 to R25, R410 to R26, R411 to R27, R412 to R28, R413 to R29, R414 to R30, R415 to R31, R416 to R32, R417 to R33, R418 to R34, R419 to R35, R420 to R36, R430 to R37, R421 to R38, R422 to R39, R423 to R40, R424 to R41, R425 to R42, R426 to R43, R427 to R44, R428 to R45, R429 to R46, TP401 to TP13, TP402 to TP14, TP403 to TP15, U301 to U4, U401 to U5

Commit message: update
Changed lines of the file:
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@@
 		(fields_autoplaced yes)
 		(property "Reference" "U5"
-			(at 241.3 20.32 0)
+			(at 241.3 12.7 0)
 			(effects
 				(font
@@
 		)
 		(property "Value" "MT41K256M16TW-107_P"
-			(at 241.3 22.86 0)
+			(at 241.3 15.24 0)
 			(effects
 				(font
@@
 		)
 		(property "PARTREV" "P"
-			(at 241.3 81.28 0)
+			(at 241.3 17.78 0)
 			(effects
 				(font
 					(size 1.27 1.27)
 				)
-				(justify bottom)
 			)
 		)
 		(property "STANDARD" "IPC-7351B"
-			(at 241.3 81.28 0)
+			(at 241.3 20.32 0)
 			(effects
 				(font
 					(size 1.27 1.27)
 				)
-				(justify bottom)
 			)
 		)
 		(property "MAXIMUM_PACKAGE_HEIGHT" "1.20mm"
-			(at 241.3 81.28 0)
+			(at 241.3 22.86 0)
 			(effects
 				(font
 					(size 1.27 1.27)
 				)
-				(justify bottom)
 			)
 		)

Commit message: update
Parts:
- removed C82, C97: 1uF, lib:C_0402_small, symbol Device:C
- removed TP13, TP14, TP15: TestPoint, lib:TP_0.5, symbol Connector:TestPoint
- added C1, C2, C3: 100nF, lib:C_0402_small, symbol Device:C
Connections:
- net GND: now also C1.1, C2.1, C3.1
- net VDD_DDR: now also C1.2, C2.2, C3.2
- no-connect marks 0 -> 3
Other:
- note added: "To connect to VDD_DDR power plane"
- moved on the sheet: C105, C83, C84
