File: PCB/DDR.kicad_sch (KiCad schematic)
At the start: 62 parts, among them U4 STM32MP157FABx, U5 MT41K256M16TW-107_P

Commit message: pcb_update
Parts:
- R17: Field6 (none) -> 1%
- R18: TOL (none) -> 1%
Changed lines of the file:
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@@
 	)
 	(junction
-		(at 360.68 213.36)
-		(diameter 0)
-		(color 0 0 0 0)
-	)
-	(junction
-		(at 349.25 227.33)
-		(diameter 0)
-		(color 0 0 0 0)
-	)
-	(junction
 		(at 336.55 162.56)
 		(diameter 0)
@@
 	)
 	(junction
-		(at 349.25 245.11)
-		(diameter 0)
-		(color 0 0 0 0)
-	)
-	(junction
 		(at 336.55 127)
 		(diameter 0)
@@
 	(wire
 		(pts
-			(xy 337.82 227.33) (xy 349.25 227.33)
-		)
-		(stroke
-			(width 0)
-			(type default)
-		)
-	)
-	(wire
-		(pts
 			(xy 349.25 245.11) (xy 360.68 245.11)
 		)
@@
 	(wire
 		(pts
-			(xy 337.82 213.36) (xy 360.68 213.36)
-		)
-		(stroke
-			(width 0)
-			(type default)
-		)
-	)
-	(wire
-		(pts
 			(xy 336.55 162.56) (xy 331.47 162.56)
 		)
@@
 	(wire
 		(pts
-			(xy 337.82 245.11) (xy 349.25 245.11)
-		)
-		(stroke
-			(width 0)
-			(type default)
-		)
-	)
-	(wire
-		(pts
 			(xy 311.15 74.93) (xy 311.15 73.66)
 		)
@@
 		(polyline
 			(pts
-				(xy 167.64 140.97) (xy 167.64 157.48) (xy 175.26 157.48) (xy 175.26 140.97)
+				(xy 194.31 73.66) (xy 214.63 73.66) (xy 214.63 133.35) (xy 194.31 133.35)
 			)
 			(stroke
@@
 		(polyline
 			(pts
-				(xy 194.31 73.66) (xy 214.63 73.66) (xy 214.63 133.35) (xy 194.31 133.35)
+				(xy 167.64 140.97) (xy 167.64 157.48) (xy 175.26 157.48) (xy 175.26 140.97)
 			)
 			(stroke
@@
 		(on_board yes)
 		(dnp no)
-		(fields_autoplaced yes)
 		(property "Reference" "R18"
 			(at 274.32 83.8199 0)
@@
 			)
 		)
+		(property "TOL" "1%"
+			(at 275.336 88.9 0)
+			(effects
+				(font
+					(size 1.27 1.27)
+				)
+			)
+		)
 		(pin "1"
 		)
@@
 		(on_board yes)
 		(dnp no)
-		(fields_autoplaced yes)
 		(property "Reference" "R17"
 			(at 172.72 144.7799 0)
@@
 			)
 		)
+		(property "Field6" "1%"
+			(at 173.736 149.352 0)
+			(effects
+				(font
+					(size 1.27 1.27)
+				)
+			)
+		)
