File: PCB/IO_Perph_Conn.kicad_sch (KiCad schematic)
At the start: 17 parts, among them U301 STM32MP157FABx, Y601 NX2012SA-32.768K

Commit message: die_length UPDATE
Parts:
- U301: footprint Package_BGA:ST_LFBGA-354_16x16mm_Layout19x19_P0.8mm -> lib:ST_LFBGA-354_16x16mm_Layout19x19_P0.8mm
Changed lines of the file:
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@@
 			)
 		)
-		(property "Footprint" "Package_BGA:ST_LFBGA-354_16x16mm_Layout19x19_P0.8mm"
+		(property "Footprint" "lib:ST_LFBGA-354_16x16mm_Layout19x19_P0.8mm"
 			(at 28.448 240.284 0)
 			(effects
@@
 			)
 		)
-		(property "Footprint" "Package_BGA:ST_LFBGA-354_16x16mm_Layout19x19_P0.8mm"
+		(property "Footprint" "lib:ST_LFBGA-354_16x16mm_Layout19x19_P0.8mm"
 			(at -70.612 213.614 0)
 			(effects

Commit message: 0402 cap update footprint
Parts:
- C601, C602: footprint Capacitor_SMD:C_0402_1005Metric -> lib:C_0402_small
Changed lines of the file:
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@@
 			)
 		)
-		(property "Footprint" "Capacitor_SMD:C_0402_1005Metric"
+		(property "Footprint" "lib:C_0402_small"
 			(at 145.7452 77.47 0)
 			(effects
@@
 			)
 		)
-		(property "Footprint" "Capacitor_SMD:C_0402_1005Metric"
+		(property "Footprint" "lib:C_0402_small"
 			(at 145.7452 100.33 0)
 			(effects
