File: PCB/MPU_PWR.kicad_sch (KiCad schematic)
At the start: 50 parts, among them U301 STM32MP157FABx

Commit message: PCB_UPDATE
Parts:
- renumbered C301 to C31, C302 to C32, C303 to C33, C304 to C34, C1 to C35, C2 to C36, C3 to C37, C4 to C38, C5 to C39, C305 to C40, C306 to C41, C307 to C42, C308 to C43, C309 to C44, C310 to C45, C311 to C46, C312 to C47, C313 to C48, C314 to C49, C315 to C50, C316 to C51, C317 to C52, C318 to C53, C319 to C54, C6 to C55, C7 to C56, C320 to C57, C321 to C58, C322 to C59, C323 to C60, C324 to C61, C325 to C62, C8 to C63, C9 to C64, C326 to C65, C327 to C66, C328 to C67, C329 to C68, C330 to C69, C331 to C70, C332 to C71, C333 to C72, C334 to C73, C335 to C74, C336 to C75, C337 to C76, C338 to C77, C339 to C78, L301 to L6, U301 to U4

Commit message: update
Parts:
- removed C35, C36, C37: 1uF, lib:C_0402_small, symbol Device:C

Commit message: pcb_update
Changed lines of the file:
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@@
 	)
 	(junction
-		(at 22.86 228.6)
-		(diameter 0)
-		(color 0 0 0 0)
-	)
-	(junction
 		(at 40.64 228.6)
 		(diameter 0)
@@
 	)
 	(junction
-		(at 22.86 234.95)
-		(diameter 0)
-		(color 0 0 0 0)
-	)
-	(junction
 		(at 85.09 214.63)
 		(diameter 0)
@@
 	)
 	(junction
-		(at 22.86 74.93)
-		(diameter 0)
-		(color 0 0 0 0)
-	)
-	(junction
 		(at 168.91 186.69)
 		(diameter 0)
@@
 	)
 	(junction
-		(at 40.64 234.95)
-		(diameter 0)
-		(color 0 0 0 0)
-	)
-	(junction
 		(at 168.91 227.33)
 		(diameter 0)
@@
 	)
 	(junction
-		(at 40.64 68.58)
-		(diameter 0)
-		(color 0 0 0 0)
-	)
-	(junction
 		(at 40.64 190.5)
 		(diameter 0)
@@
 	)
 	(junction
-		(at 40.64 81.28)
-		(diameter 0)
-		(color 0 0 0 0)
-	)
-	(junction
 		(at 137.16 121.92)
 		(diameter 0)
@@
 	)
 	(junction
-		(at 40.64 74.93)
-		(diameter 0)
-		(color 0 0 0 0)
-	)
-	(junction
 		(at 256.54 119.38)
 		(diameter 0)
@@
 	)
 	(junction
-		(at 22.86 81.28)
-		(diameter 0)
-		(color 0 0 0 0)
-	)
-	(junction
 		(at 40.64 215.9)
 		(diameter 0)
@@
 	)
 	(junction
-		(at 40.64 241.3)
-		(diameter 0)
-		(color 0 0 0 0)
-	)
-	(junction
 		(at 40.64 146.05)
 		(diameter 0)
@@
 	)
 	(junction
-		(at 22.86 68.58)
-		(diameter 0)
-		(color 0 0 0 0)
-	)
-	(junction
 		(at 256.54 132.08)
 		(diameter 0)
@@
 	(wire
 		(pts
-			(xy 40.64 68.58) (xy 40.64 74.93)
-		)
-		(stroke
-			(width 0)
-			(type default)
-		)
-	)
-	(wire
-		(pts
 			(xy 168.91 247.65) (xy 168.91 250.19)
 		)
@@
 	(wire
 		(pts
-			(xy 22.86 74.93) (xy 27.94 74.93)
-		)
-		(stroke
-			(width 0)
-			(type default)
-		)
-	)
-	(wire
-		(pts
 			(xy 256.54 101.6) (xy 256.54 104.14)
 		)
@@
 	(wire
 		(pts
-			(xy 22.86 74.93) (xy 22.86 81.28)
+			(xy 22.86 60.96) (xy 22.86 87.63)
 		)
 		(stroke
@@
 	(wire
 		(pts
-			(xy 22.86 60.96) (xy 22.86 68.58)
-		)
-		(stroke
-			(width 0)
-			(type default)
-		)
-	)
-	(wire
-		(pts
 			(xy 22.86 184.15) (xy 27.94 184.15)
 		)
@@
 	(wire
 		(pts
-			(xy 40.64 228.6) (xy 40.64 234.95)
+			(xy 40.64 228.6) (xy 40.64 243.84)
 		)
 		(stroke
@@
 	(wire
 		(pts
-			(xy 22.86 81.28) (xy 27.94 81.28)
-		)
-		(stroke
-			(width 0)
-			(type default)
-		)
-	)
-	(wire
-		(pts
 			(xy 40.64 158.75) (xy 35.56 158.75)
 		)
@@
 	(wire
 		(pts
-			(xy 22.86 68.58) (xy 27.94 68.58)
-		)
-		(stroke
-			(width 0)
-			(type default)
-		)
-	)
-	(wire
-		(pts
 			(xy 256.54 213.36) (xy 254 213.36)
 		)
@@
 	(wire
 		(pts
-			(xy 40.64 68.58) (xy 35.56 68.58)
-		)
-		(stroke
-			(width 0)
-			(type default)
-		)
-	)
-	(wire
-		(pts
 			(xy 22.86 203.2) (xy 27.94 203.2)
 		)
@@
 	(wire
 		(pts
-			(xy 22.86 241.3) (xy 27.94 241.3)
-		)
-		(stroke
-			(width 0)
-			(type default)
-		)
-	)
-	(wire
-		(pts
-			(xy 40.64 234.95) (xy 35.56 234.95)
-		)
-		(stroke
-			(width 0)
-			(type default)
-		)
-	)
-	(wire
-		(pts
-			(xy 40.64 241.3) (xy 40.64 243.84)
-		)
-		(stroke
-			(width 0)
-			(type default)
-		)
-	)
-	(wire
-		(pts
 			(xy 168.91 191.77) (xy 171.45 191.77)
 		)
@@
 	(wire
 		(pts
-			(xy 22.86 228.6) (xy 22.86 234.95)
-		)
-		(stroke
-			(width 0)
-			(type default)
-		)
-	)
-	(wire
-		(pts
 			(xy 40.64 127) (xy 35.56 127)
 		)
@@
 	(wire
 		(pts
-			(xy 40.64 60.96) (xy 40.64 68.58)
+			(xy 40.64 60.96) (xy 40.64 87.63)
 		)
 		(stroke
@@
 	(wire
 		(pts
-			(xy 40.64 81.28) (xy 35.56 81.28)
-		)
-		(stroke
-			(width 0)
-			(type default)
-		)
-	)
-	(wire
-		(pts
 			(xy 153.67 252.73) (xy 144.78 252.73)
 		)
@@
 	(wire
 		(pts
-			(xy 40.64 241.3) (xy 35.56 241.3)
-		)
-		(stroke
-			(width 0)
-			(type default)
-		)
-	)
-	(wire
-		(pts
 			(xy 256.54 53.34) (xy 254 53.34)
 		)
@@
 	(wire
 		(pts
-			(xy 22.86 68.58) (xy 22.86 74.93)
-		)
-		(stroke
-			(width 0)
-			(type default)
-		)
-	)
-	(wire
-		(pts
 			(xy 256.54 132.08) (xy 256.54 134.62)
 		)
@@
 	(wire
 		(pts
-			(xy 22.86 234.95) (xy 22.86 241.3)
-		)
-		(stroke
-			(width 0)
-			(type default)
-		)
-	)
-	(wire
-		(pts
 			(xy 22.86 87.63) (xy 27.94 87.63)
 		)
@@
 	(wire
 		(pts
-			(xy 40.64 74.93) (xy 35.56 74.93)
-		)
-		(stroke
-			(width 0)
-			(type default)
-		)
-	)
-	(wire
-		(pts
 			(xy 35.56 93.98) (xy 40.64 93.98)
 		)
@@
 	(wire
 		(pts
-			(xy 22.86 234.95) (xy 27.94 234.95)
-		)
-		(stroke
-			(width 0)
-			(type default)
-		)
-	)
-	(wire
-		(pts
 			(xy 256.54 66.04) (xy 256.54 68.58)
 		)
@@
 	(wire
 		(pts
-			(xy 40.64 74.93) (xy 40.64 81.28)
-		)
-		(stroke
-			(width 0)
-			(type default)
-		)
-	)
-	(wire
-		(pts
 			(xy 256.54 240.03) (xy 254 240.03)
 		)
@@
 	(wire
 		(pts
-			(xy 40.64 81.28) (xy 40.64 87.63)
-		)
-		(stroke
-			(width 0)
-			(type default)
-		)
-	)
-	(wire
-		(pts
 			(xy 256.54 144.78) (xy 256.54 147.32)
 		)
@@
 	(wire
 		(pts
-			(xy 40.64 234.95) (xy 40.64 241.3)
-		)
-		(stroke
-			(width 0)
-			(type default)
-		)
-	)
-	(wire
-		(pts
 			(xy 168.91 229.87) (xy 168.91 232.41)
 		)
@@
 		)
 		(stroke
-			(width 0)
-			(type default)
-		)
-	)
-	(wire
-		(pts
-			(xy 22.86 81.28) (xy 22.86 87.63)
-		)
-		(stroke
