File: PCB/PWR.kicad_sch (KiCad schematic)
At the start: 41 parts, among them Q1 CSD23381F4, U3 STPMIC1APQR

Commit message: update
Parts:
- added TP1, TP2: TestPoint, lib:TP_0.5, symbol Connector:TestPoint
Connections:
- net 1V8: now reaches C25.2, U3.21 (LDO6OUT)
- net 1V8: now also TP2.1
- net 2V8: now reaches C20.2, U3.23 (LDO1OUT)
- net 2V8: now also TP1.1
Other:
- note added: "120mA LDO max"
- note added: "150mA LDO max"
- note added: "350mA LDO max"
- note added: "50mA LDO max"

Commit message: pcb_update
Other:
- note added: "Caution: VDD3V3_USBHS must not be present unless VDDA1V8_REG is present, otherwise permanent STM32MP15x lines damage can occur. It must be ensured by PMIC ranking order or with external component in case of discrete component power-supply implementation."
Changed lines of the file:
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@@
 		(comment 1 "Author: Mykola Grodskyi")
 	)
+	(text "Caution: VDD3V3_USBHS must not be present unless VDDA1V8_REG is present, otherwise permanent\nSTM32MP15x lines damage can occur. It must be ensured by PMIC ranking order or with\nexternal component in case of discrete component power-supply implementation."
+		(exclude_from_sim no)
+		(at 237.998 101.346 0)
+		(effects
+			(font
+				(size 1.27 1.27)
+			)
+		)
+	)
 	(text "150mA LDO max\n"
 		(exclude_from_sim no)
@@
 			"AAAAAAAAAAAAAAAAAAAAAAAAAAAAAAAAAAAAAAAAAAAAAAAAAAAAAAAAAAAAAAAAAAAAAAAAAAAA"
 			"AAAAAAAAAAAAAAAAAAAAAAAAAAAAAAAAAAAAAAAAAAAAAAAAAAAAAAAAAAAAAAAAAAAAAAAAAAAA"
+			"AAAAAAAAAAAAAAAAAAAAAAAAAAAAAAAAAAAAAAAAAAAAAAAAAAAAAAAAAAAAAAAAAAAAAAAAAAAA"
+			"AAAAAAAAAAAAAAAAAAAAAAAAAAAAAAAAAAAAAAAAAAAAAAAAAAAAAAAAAAAAAAAAAAAAAAAAAAAA"
+			"AAAAAAAAAAAAAAAAAAAAAAAAAAAAAAAAAAAAAAAAAAAAAAAAAAAAAAAAAAAAAAAAAAAAAAAAAAAA"
+			"AAAAAAAAAAAAAAAAAAAAAAAAAAAAAAAAAAAAAAAAAAAAAAAAAAAAAAAAAAAAAAAAAAAAAAAAAAAA"
+			"AAAAAAAAAAAAAAAAAAAAAAAAAAAAAAAAAAAAAAAAAAAAAAAAAAAAAAAAAAAAAAAAAAAAAAAAAAAA"
+			"AAAAAAAAAAAAAAAAAAAAAAAAAAAAAAAAAAAAAAAAAAAAAAAAAAAAAAAAAAAAAAAAAAAAAAAAAAAA"
+			"AAAAAAAAAAAAAAAAAAAAAAAAAAAAAAAAAAAAAAAAAAAAAAAAAAAAAAAAAAAAAAAAAAAAAAAAAAAA"
+			"AAAAAAAAAAAAAAAAAAAAAAAAAAAAAAAAAAAAAAAAAAAAAAAAAAAAAAAAAAAAAAAAAAAAAAAAAAAA"
+			"AAAAAAAAAAAAAAAAAAAAAAAAAAAAAAAAAAAAAAAAAAAAAAAAAAAAAAAAAAAAAAAAAAAAAAAAAAAA"
+			"AAAAAAAAAAAAAAAAAAAAAAAAAAAAAAAAAAAAAAAAAAAAAAAAAAAAAAAAAAAAAAAAAAAAAAAAAAAA"
+			"AAAAAAAAAAAAAAAAAAAAAAAAAAAAAAAAAAAAAAAAAAAAAAAAAAAAAAAAAAAAAAAAAAAAAAAAAAAA"
+			"AAAAAAAAAAAAAAAAAAAAAAAAAAAAAAAAAAAAAAAAAAAAAAAAAAAAAAAAAAAAAAAAAAAAAAAAAAAA"
+			"AAAAAAAAAAAAAAAAAAAAAAAAAAAAAAAAAAAAAAAAAAAAAAAAAAAAAAAAAAAAAAAAAAAAAAAAAAAA"
+			"AAAAAAAAAAAAAAAAAAAAAAAAAAAAAAAAAAAAAAAAAAAAAAAAAAAAAAAAAAAAAAAAAAAAAAAAAAAA"
+			"AAAAAAAAAAAAAAAAAAAAAAAAAAAAAAAAAAAAAAAAAAAAAAAAAAAAAAAAAAAAAAAAAAAAAAAAAAAA"
+			"AAAAAAAAAAAAAAAAAAAAAAAAAAAAAAAAAAAAAAAAAAAAAAAAAAAAAAAAAAAAAAAAAAAAAAAAAAAA"
+			"AAAAAAAAAAAAAAAAAAAAAAAAAAAAAAAAAAAAAAAAAAAAAAAAAAAAAAAAAAAAAAAAAAAAAAAAAAAA"
+			"AAAAAAAAAAAAAAAAAAAAAAAAAAAAAAAAAAAAAAAAAAAAAAAAAAAAAAAAAAAAAAAAAAAAAAAAAAAA"
+			"AAAAAAAAAAAAAAAAAAAAAAAAAAAAAAAAAAAAAAAAAAAAAAAAAAAAAAAAAAAAAAAAAAAAAAAAAAAA"
+			"AAAAAAAAAAAAAAAAAAAAAAAAAAAAAAAAAAAAAAAAAAAAAAAAAAAAAAAAAAAAAAAAAAAAAAAAAAAA"
+			"AAAAAAAAAAAAAAAAAAAAAAAAAAAAAAAAAAAAAAAAAAAAAAAAAAAAAAAAAAAAAAAAAAAAAAAAAAAA"
+			"AAAAAAAAAAAAAAAAAAAAAAAAAAAAAAAAAAAAAAAAAAAAAAAAAAAAAAAAAAAAAAAAAAAAAAAAAAAA"
+			"AAAAAAAAAAAAAAAAAAAAAAAAAAAAAAAAAAAAAAAAAAAAAAAAAAAAAAAAAAAAAAAAAAAAAAAAAAAA"
+			"AAAAAAAAAAAAAAAAAAAAAAAAAAAAAAAAAAAAAAAAAAAAAAAAAAAAAAAAAAAAAAAAAAAAAAAAAAAA"
+			"AAAAAAAAAAAAAAAAAAAAAAAAAAAAAAAAAAAAAAAAAAAAAAAAAAAAAAAAAAAAAAAAAAAAAAAAAAAA"
+			"AAAAAAAAAAAAAAAAAAAAAAAAAAAAAAAAAAAAAAAAAAAAAAAAAAAAAAAAAAAAAAAAAAAAAAAAAAAA"
+			"AAAAAAAAAAAAAAAAAAAAAAAAAAAAAAAAAAAAAAAAAAAAAAAAAAAAAAAAAAAAAAAAAAAAAAAAAAAA"
+			"AAAAAAAAAAAAAAAAAAAAAAAAAAAAAAAAAAAAAAAAAAAAAAAAAAAAAAAAAAAAAAAAAAAAAAAAAAAA"
+			"AAAAAAAAAAAAAAAAAAAAAAAAAAAAAAAAAAAAAAAAAAAAAAAAAAAAAAAAAAAAAAAAAAAAAAAAAAAA"
+			"AAAAAAAAAAAAAAAAAAAAAAAAAAAAAAAAAAAAAAAAAAAAAAAAAAAAAAAAAAAAAAAAAAAAAAAAAAAA"
+			"AAAAAAAAAAAAAAAAAAAAAAAAAAAAAAAAAAAAAAAAAAAAAAAAAAAAAAAAAAAAAAAAAAAAAAAAAAAA"
+			"AAAAAAAAAAAAAAAAAAAAAAAAAAAAAAAAAAAAAAAAAAAAAAAAAAAAAAAAAAAAAAAAAAAAAAAAAAAA"
+			"AAAAAAAAAAAAAAAAAAAAAAAAAAAAAAAAAAAAAAAAAAAAAAAAAAAAAAAAAAAAAAAAAAAAAAAAAAAA"
+			"AAAAAAAAAAAAAAAAAAAAAAAAAAAAAAAAAAAAAAAAAAAAAAAAAAAAAAkJCShmb250CgkJCQkJCQkJ"
+			"KHNpemUgMS4yNyAxLjI3KQoJCQkJCQkJKQoJCQkJCQkpCgkJCQkJKQoJCQkJKQoJCQkJKHBpbiBw"
+			"YXNzaXZlIGxpbmUKCQkJCQkoYXQgNTQuNjEgLTQ4LjI2IDE4MCkKCQkJCQkobGVuZ3RoIDUuMDgp"
+			"CgkJCQkJKG5hbWUgIlZTUyIKCQkJCQkJKGVmZmVjdHMKCQkJCQkJCShmb250CgkJCQkJCQkJKHNp"
+			"emUgMS4yNyAxLjI3KQoJCQkJCQkJKQoJCQkJCQkpCgkJCQkJKQoJCQkJCShudW1iZXIgIkY5IgoJ"
+			"CQkJCQkoZWZmZWN0cwoJCQkJCQkJKGZvbnQKCQkJCQkJCQkoc2l6ZSAxLjI3IDEuMjcpCgkJCQkJ"
+			"CQkpCgkJCQkJCSkKCQkJCQkpCgkJCQkpCgkJCQkocGluIHBhc3NpdmUgbGluZQoJCQkJCShhdCA1"
+			"NC42MSAtNTAuOCAxODApCgkJCQkJKGxlbmd0aCA1LjA4KQoJCQkJCShuYW1lICJWU1MiCgkJCQkJ"
+			"CShlZmZlY3RzCgkJCQkJCQkoZm9udAoJCQkJCQkJCShzaXplIDEuMjcgMS4yNykKCQkJCQkJCSkK"
+			"CQkJCQkJKQoJCQkJCSkKCQkJCQkobnVtYmVyICJGNyIKCQkJCQkJKGVmZmVjdHMKCQkJCQkJCShm"
+			"b250CgkJCQkJCQkJKHNpemUgMS4yNyAxLjI3KQoJCQkJCQkJKQoJCQkJCQkpCgkJCQkJKQoJCQkJ"
+			"KQoJCQkJKHBpbiBwYXNzaXZlIGxpbmUKCQkJCQkoYXQgNTQuNjEgLTUzLjM0IDE4MCkKCQkJCQko"
+			"bGVuZ3RoIDUuMDgpCgkJCQkJKG5hbWUgIlZTUyIKCQkJCQkJKGVmZmVjdHMKCQkJCQkJCShmb250"
+			"CgkJCQkJCQkJKHNpemUgMS4yNyAxLjI3KQoJCQkJCQkJKQoJCQkJCQkpCgkJCQkJKQoJCQkJCShu"
+			"dW1iZXIgIkY1IgoJCQkJCQkoZWZmZWN0cwoJCQkJCQkJKGZvbnQKCQkJCQkJCQkoc2l6ZSAxLjI3"
+			"IDEuMjcpCgkJCQkJCQkpCgkJCQkJCSkKCQkJCQkpCgkJCQkpCgkJCQkocGluIHBhc3NpdmUgbGlu"
+			"ZQoJCQkJCShhdCA1NC42MSAtNTUuODggMTgwKQoJCQkJCShsZW5ndGggNS4wOCkKCQkJCQkobmFt"
+			"ZSAiVlNTIgoJCQkJCQkoZWZmZWN0cwoJCQkJCQkJKGZvbnQKCQkJCQkJCQkoc2l6ZSAxLjI3IDEu"
+			"MjcpCgkJCQkJCQkpCgkJCQkJCSkKCQkJCQkpCgkJCQkJKG51bWJlcgAAAAAAAAAAAAAAAAAAAAAA"
+			"AAAAAAAAAAAAAAAAAAAAAAAAAAAAAAAAAAAAAAAAAAAAAAAAAAAAAAAAAAAAAAAAAAAAAAAAAAAA"
+			"AAAAAAAAAAAAAAAAAAAAAAAAAAAAAAAAAAAAAAAAAAAAAAAAAAAAAAAAAAAAAAAAAAAAAAAAAAAA"
+			"AAAAAAAAAAAAAAAAAAAAAAAAAAAAAAAAAAAAAAAAAAAAAAAAAAAAAAAAAAAAAAAAAAAAAAAAAAAA"
+			"AAAAAAAAAAAAAAAAAAAAAAAAAAAAAAAAAAAAAAAAAAAAAAAAAAAAAAAAAAAAAAAAAAAAAAAAAAAA"
+			"AAAAAAAAAAAAAAAAAAAAAAAAAAAAAAAAAAAAAAAAAAAAAAAAAAAAAAAAAAAAAAAAAAAAAAAAAAAA"
+			"AAAAAAAAAAAAAAAAAAAAAAAAAAAAAAAAAAAAAAAAAAAAAAAAAAAAAAAAAAAAAAAAAAAAAAAAAAAA"
+			"AAAAAAAAAAAAAAAAAAAAAAAAAAAAAAAAAAAAAAAAAAAAAAAAAAAAAAAAAAAAAAAAAAAAAAAAAAAA"
+			"AAAAAAAAAAAAAAAAAAAAAAAAAAAAAAAAAAAAAAAAAAAAAAAAAAAAAAAAAAAAAAAAAAAAAAAAAAAA"
+			"AAAAAAAAAAAAAAAAAAAAAAAAAAAAAAAAAAAAAAAAAAAAAAAAAAAAAAAAAAAAAAAAAAAAAAAAAAAA"
+			"AAAAAAAAAAAAAAAAAAAAAAAAAAAAAAAAAAAAAAAAAAAAAAAAAAAAAAAAAAAAAAAAAAAAAAAAAAAA"
+			"AAAAAAAAAAAAAAAAAAAAAAAAAAAAAAAAAAAAAAAAAAAAAAAAAAAAAAAAAAAAAAAAAAAAAAAAAAAA"
+			"AAAAAAAAAAAAAAAAAAAAAAAAAAAAAAAAAAAAAAAAAAAAAAAAAAAAAAAAAAAAAAAAAAAAAAAAAAAA"
+			"AAAAAAAAAAAAAAAAAAAAAAAAAAAAAAAAAAAAAAAAAAAAAAAAAAAAAAAAAAAAAAAAAAAAAAAAAAAA"
+			"AAAAAAAAAAAAAAAAAAAAAAAAAAAAAAAAAAAAAAAAAAAAAAAAAAAAAAAAAAAAAAAAAAAAAAAAAAAA"
+			"AAAAAAAAAAAAAAAAAAAAAAAAAAAAAAAAAAAAAAAAAAAAAAAAAAAAAAAAAAAAAAAAAAAAAAAAAAAA"
+			"AAAAAAAAAAAAAAAAAAAAAAAAAAAAAAAAAAAAAAAAAAAAAAAAAAAAAAAAAAAAAAAAAAAAAAAAAAAA"
+			"AAAAAAAAAAAAAAAAAAAAAAAAAAAAAAAAAAAAAAAAAAAAAAAAAAAAAAAAAAAAAAAAAAAAAAAAAAAA"
+			"AAAAAAAAAAAAAAAAAAAAAAAAAAAAAAAAAAAAAAAAAAAAAAAAAAAAAAAAAAAAAAAAAAAAAAAAAAAA"
+			"AAAAAAAAAAAAAAAAAAAAAAAAAAAAAAAAAAAAAAAAAAAAAAAAAAAAAAAAAAAAAAAAAAAAAAAAAAAA"
+			"AAAAAAAAAAAAAAAAAAAAAAAAAAAAAAAAAAAAAAAAAAAAAAAAAAAAAAAAAAAAAAAAAAAAAAAAAAAA"
