File: PCB/PWR.kicad_sch (KiCad schematic)
At the start: 47 parts, among them Q201 DMG1013T-7, U201 TPS62840DLCR, U202 STPMIC1APQR

Commit message: UPDATE
Parts:
- removed D201: MSP3V3-M3/89A, Diode_SMD:D_MicroSMP_KA, symbol PTVS3V3S1UR:PTVS3V3S1UR
- added D3: DF2S5M4CT,L3F, Diode_SMD:D_SOD-882, symbol PTVS3V3S1UR:PTVS3V3S1UR
Connections:
- net GND: now also D3.2
- net at C203.2, S2.1, U202.17 (~{PONKEY}): now also D3.1

Commit message: PCB_UPDATE
Other:
- note added: "CHECKED 2.0 MG"
- note added: "only PA0"
- note added: "only PC13"
Changed lines of the file:
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@@
+		)
+	)
+	(text "only PC13\n"
+		(exclude_from_sim no)
+		(at 210.058 205.232 0)
+		(effects
+			(font
+				(size 1.27 1.27)
+			)
 		)
 	)
@@
 		)
 	)
+	(text "CHECKED 2.0 MG\n"
+		(exclude_from_sim no)
+		(at 175.514 139.7 0)
+		(effects
+			(font
+				(size 12.7 12.7)
+				(color 97 255 51 1)
+			)
+		)
+	)
 	(text "120mA LDO max\n"
 		(exclude_from_sim no)
@@
 		(effects
 			(font
+				(size 1.27 1.27)
+			)
+		)
+	)
+	(text "only PA0\n\n"
+		(exclude_from_sim no)
+		(at 267.97 235.204 0)
+		(effects
+			(font
