File: PCB/RCC_BOOT_RST_DEBUG.kicad_sch (KiCad schematic)
At the start: 38 parts, among them J701 FTSH-107-01-L-DV-K-A, U301 STM32MP157FABx, U701 HSP051-4M10, U702 HSP051-4M10, Y701 ECS-2520MVQ-240

Commit message: looks like i fixed DDR
Parts:
- removed R702, R703: 0, Resistor_SMD:R_0402_1005Metric, symbol Device:R
Connections:
- net GND: now also U301.T15 (BYPASS_REG1V8)

Commit message: 0402 cap update footprint
Parts:
- C701, C702, C703, C704, C705: footprint Capacitor_SMD:C_0402_1005Metric -> lib:C_0402_small
Changed lines of the file:
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@@
 			)
 		)
-		(property "Footprint" "Capacitor_SMD:C_0402_1005Metric"
+		(property "Footprint" "lib:C_0402_small"
 			(at 80.9752 33.02 0)
 			(effects
@@
 			)
 		)
-		(property "Footprint" "Capacitor_SMD:C_0402_1005Metric"
+		(property "Footprint" "lib:C_0402_small"
 			(at 136.1948 125.73 0)
 			(effects
@@
 			)
 		)
-		(property "Footprint" "Capacitor_SMD:C_0402_1005Metric"
+		(property "Footprint" "lib:C_0402_small"
 			(at 296.2148 52.07 0)
 			(effects
@@
 			)
 		)
-		(property "Footprint" "Capacitor_SMD:C_0402_1005Metric"
+		(property "Footprint" "lib:C_0402_small"
 			(at 290.83 32.0548 0)
 			(effects
@@
 			)
 		)
-		(property "Footprint" "Capacitor_SMD:C_0402_1005Metric"
+		(property "Footprint" "lib:C_0402_small"
 			(at 261.9248 52.07 0)
 			(effects
