File: PCB/RCC_BOOT_RST_DEBUG.kicad_sch (KiCad schematic)
At the start: 26 parts, among them J701 FTSH-107-01-L-DV-K-A, U301 STM32MP157FABx, U701 HSP051-4M10, U702 HSP051-4M10, Y701 ECS-2520MVQ-240

Commit message: PCB_UPDATE
Parts:
- renumbered C701 to C112, C702 to C113, C703 to C114, C704 to C115, C705 to C116, D5 to D7, J701 to J2, R701 to R58, R2 to R59, R3 to R60, R1 to R61, R706 to R62, R709 to R63, R710 to R64, R711 to R65, R712 to R66, R713 to R67, R714 to R68, R715 to R69, S701 to S5, TP701 to TP21, TP702 to TP22, U301 to U4, U701 to U8, U702 to U9, Y701 to Y2

Commit message: update
Other:
- note added: "powering from st link is wrong"
Changed lines of the file:
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@@
 		(comment 1 "Author: Mykola Grodskyi")
+	)
+	(text "powering from st link is wrong\n"
+		(exclude_from_sim no)
+		(at 380.492 83.82 0)
+		(effects
+			(font
+				(size 1.27 1.27)
+			)
+		)
 	)
 	(junction

Commit message: update
Parts:
- removed D7: MSP3V3-M3/89A, Diode_SMD:D_MicroSMP_KA, symbol PTVS3V3S1UR:PTVS3V3S1UR
Other:
- note removed: "powering from st link is wrong"

Commit message: pcb_update
Parts:
- added TP25, TP26, TP27, TP29, TP30: TestPoint, lib:TP_0.5, symbol Connector:TestPoint
Connections:
- net GND: now also TP30.1
- net VDD: now also TP29.1; no longer C115.1
- net at R60.1, R63.1, U4.K4 (BOOT1): now also TP26.1
- net at R68.1, Y2.4 (VDD): now also C115.1
- net at R59.1, R64.2, U4.K1 (BOOT0): now also TP27.1
- net at R61.1, R62.2, U4.L2 (BOOT2): now also TP25.1
Other:
- moved on the sheet: C115, R68
