File: PCB/WIFI_BLE.kicad_sch (KiCad schematic)
At the start: 25 parts, among them J901 73412-0110, U901 LBEE5PK2AE-771

Commit message: 0402 cap update footprint
Parts:
- C901, C904, C905: footprint Capacitor_SMD:C_0402_1005Metric -> lib:C_0402_small
Changed lines of the file:
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@@
 			)
 		)
-		(property "Footprint" "Capacitor_SMD:C_0402_1005Metric"
+		(property "Footprint" "lib:C_0402_small"
 			(at 246.6848 67.31 0)
 			(effects
@@
 			)
 		)
-		(property "Footprint" "Capacitor_SMD:C_0402_1005Metric"
+		(property "Footprint" "lib:C_0402_small"
 			(at 246.6848 49.53 0)
 			(effects
@@
 			)
 		)
-		(property "Footprint" "Capacitor_SMD:C_0402_1005Metric"
+		(property "Footprint" "lib:C_0402_small"
 			(at 239.0648 96.52 0)
 			(effects
