File: PCB/WIFI_BLE.kicad_sch (KiCad schematic)
At the start: 25 parts, among them J901 73412-0110, U901 LBEE5PK2AE-771

Commit message: PCB_UPDATE
Parts:
- added U1: LBEE5KL1YN-814, lib:XCVR_LBEE5KL1YN-814, symbol LBEE5KL1YN-814:LBEE5KL1YN-814
Changed lines of the file:
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@@
+	)
+	(symbol
+		(lib_id "LBEE5KL1YN-814:LBEE5KL1YN-814")
+		(at 92.71 205.74 0)
+		(unit 1)
+		(exclude_from_sim no)
+		(in_bom yes)
+		(on_board yes)
+		(dnp no)
+		(fields_autoplaced yes)
+		(property "Reference" "U1"
+			(at 92.71 170.18 0)
+			(effects
+				(font
+					(size 1.27 1.27)
+				)
+			)
+		)
+		(property "Value" "LBEE5KL1YN-814"
+			(at 92.71 172.72 0)
+			(effects
+				(font
+					(size 1.27 1.27)
+				)
+			)
+		)
+		(property "Footprint" "lib:XCVR_LBEE5KL1YN-814"
+			(at 92.71 205.74 0)
+			(effects
+				(font
+					(size 1.27 1.27)
+				)
+				(justify bottom)
+				(hide yes)
+			)
+		)
+		(property "Datasheet" ""
+			(at 92.71 205.74 0)
+			(effects
+				(font
+					(size 1.27 1.27)
+				)
+				(hide yes)
+			)
+		)
+		(property "Description" ""
+			(at 92.71 205.74 0)
+			(effects
+				(font
+					(size 1.27 1.27)
+				)
+				(hide yes)
+			)
+		)
+		(property "PARTREV" "C"
+			(at 92.71 205.74 0)
+			(effects
+				(font
+					(size 1.27 1.27)
+				)
+				(justify bottom)
+				(hide yes)
+			)
+		)
+		(property "SNAPEDA_PN" "LBEE5KL1YN-814"
+			(at 92.71 205.74 0)
+			(effects
+				(font
+					(size 1.27 1.27)
+				)
+				(justify bottom)
+				(hide yes)
+			)
+		)
+		(property "MANUFACTURER" "Murata"
+			(at 92.71 205.74 0)
+			(effects
+				(font
+					(size 1.27 1.27)
+				)
+				(justify bottom)
+				(hide yes)
+			)
+		)
+		(property "MAXIMUM_PACKAGE_HEIGHT" "1.1mm"
+			(at 92.71 205.74 0)
+			(effects
+				(font
+					(size 1.27 1.27)
+				)
+				(justify bottom)
+				(hide yes)
+			)
+		)
+		(property "STANDARD" "Manufacturer Recommendations"
+			(at 92.71 205.74 0)
+			(effects
+				(font
+					(size 1.27 1.27)
+				)
+				(justify bottom)
+				(hide yes)
+			)
+		)
+		(pin "13"
+		)
+		(pin "31"
+		)
+		(pin "36"
+		)
+		(pin "6"
+		)
+		(pin "37"
+		)
+		(pin "41"
+		)
+		(pin "17"
+		)
+		(pin "18"
+		)
+		(pin "15"
+		)
+		(pin "7"
+		)
+		(pin "30"
+		)
+		(pin "16"
+		)
+		(pin "32"
+		)
+		(pin "33"
+		)
+		(pin "46"
+		)
+		(pin "9"
+		)
+		(pin "14"
+		)
+		(pin "8"
+		)
+		(pin "28"
+		)
+		(pin "10"
+		)
+		(pin "11"
+		)
+		(pin "27"
+		)
+		(pin "20"
+		)
+		(pin "22"
+		)
+		(pin "12"
+		)
+		(pin "34"
+		)
+		(pin "19"
+		)
+		(pin "5"
+		)
+		(pin "38"
+		)
+		(pin "24"
+		)
+		(pin "23"
+		)
+		(pin "21"
+		)
+		(pin "29"
+		)
+		(pin "4"
+		)
+		(pin "35"
+		)
+		(pin "44"
+		)
+		(pin "45"
+		)
+		(pin "25"
+		)
+		(pin "2"
+		)
+		(pin "39"
+		)
+		(pin "40"
+		)
+		(pin "42"
+		)
+		(pin "43"
+		)
+		(pin "26"
+		)
+		(pin "1"
+		)
+		(pin "3"
+		)
+		(instances
+			(project ""
+				(path "/65890f61-d586-475b-928a-b635a5e4e59e/7b5607bb-cf07-41c5-a9f4-2640606f574f"
+					(reference "U1")
+					(unit 1)
+				)
+			)
+		)
 	)
 	(symbol
