File: PCB/MPU_MOD.kicad_sch (KiCad schematic)
At the start: 0 parts

Commit message: PCB_UPDATE
Other:
- added sheet MODULE_CONNECTOR (MODULE_CONNECTOR.kicad_sch)
Changed lines of the file:
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@@
+	)
+	(sheet
+		(at 323.85 204.47)
+		(size 54.61 33.02)
+		(exclude_from_sim no)
+		(in_bom yes)
+		(on_board yes)
+		(dnp no)
+		(fields_autoplaced yes)
+		(stroke
+			(width 0.1524)
+			(type solid)
+		)
+		(fill
+			(color 0 0 0 0.0000)
+		)
+		(property "Sheetname" "MODULE_CONNECTOR"
+			(at 323.85 203.7584 0)
+			(effects
+				(font
+					(size 1.27 1.27)
+				)
+				(justify left bottom)
+			)
+		)
+		(property "Sheetfile" "MODULE_CONNECTOR.kicad_sch"
+			(at 323.85 238.0746 0)
+			(effects
+				(font
+					(size 1.27 1.27)
+				)
+				(justify left top)
+			)
+		)
+		(instances
+			(project "MPU_MOD"
+				(path "/65890f61-d586-475b-928a-b635a5e4e59e"
+					(page "11")
+				)
+			)
+		)
 	)
 	(sheet
