File: PCB/MPU_MOD.kicad_sch (KiCad schematic)
At the start: 0 parts

Commit message: PCB_UPDATE
Parts:
- added H1, H2, H3, H4: MountingHole_Pad, MountingHole:MountingHole_2.7mm_M2.5_Pad_Via, symbol Mechanical:MountingHole_Pad
Other:
- added sheet LCD (LCD.kicad_sch)

Commit message: PCB_UPDATE
Parts:
- renumbered H3 to H2, H2 to H3
Other:
- added sheet USB (USB.kicad_sch)
