File: PCB/LCD.kicad_sch (KiCad schematic)
At the start: 1 part, among them J4 SFV30R-4STBE1HLF

Commit message: PCB_UPDATE
Parts:
- renumbered J4 to J5
Changed lines of the file:
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@@
 		(on_board yes)
 		(dnp no)
-		(property "Reference" "#PWR0101"
+		(property "Reference" "#PWR0158"
 			(at 212.09 64.77 0)
 			(effects
@@
 			(project "MPU_MOD"
 				(path "/65890f61-d586-475b-928a-b635a5e4e59e/6d63342e-f801-4ef3-ba79-fab0475ee1d8"
-					(reference "#PWR0101")
+					(reference "#PWR0158")
 					(unit 1)
 				)
@@
 		(on_board yes)
 		(dnp no)
-		(property "Reference" "#PWR05"
+		(property "Reference" "#PWR0157"
 			(at 198.12 64.77 0)
 			(effects
@@
 			(project "MPU_MOD"
 				(path "/65890f61-d586-475b-928a-b635a5e4e59e/6d63342e-f801-4ef3-ba79-fab0475ee1d8"
-					(reference "#PWR05")
+					(reference "#PWR0157")
 					(unit 1)
 				)
@@
 		(dnp no)
 		(fields_autoplaced yes)
-		(property "Reference" "J4"
+		(property "Reference" "J5"
 			(at 181.61 87.6299 0)
 			(effects
@@
 			(project ""
 				(path "/65890f61-d586-475b-928a-b635a5e4e59e/6d63342e-f801-4ef3-ba79-fab0475ee1d8"
-					(reference "J4")
+					(reference "J5")
 					(unit 1)
 				)
@@
 		(on_board yes)
 		(dnp no)
-		(property "Reference" "#PWR04"
+		(property "Reference" "#PWR0159"
 			(at 213.36 129.54 0)
 			(effects
@@
 			(project "MPU_MOD"
 				(path "/65890f61-d586-475b-928a-b635a5e4e59e/6d63342e-f801-4ef3-ba79-fab0475ee1d8"
-					(reference "#PWR04")
+					(reference "#PWR0159")
 					(unit 1)
 				)

Commit message: update
Parts:
- removed J5: SFV30R-4STBE1HLF, lib:AMPHENOL_SFV30R-4STBE1HLF, symbol SFV30R-4STBE1HLF:SFV30R-4STBE1HLF
- added C35: 1uF, lib:C_0402_small, symbol Device:C
- added C4, C5, C6: 0.47uF, lib:C_0402_small, symbol Device:C
- added C7, C8: 100nF, lib:C_0402_small, symbol Device:C
- added C9: 4.7uF, lib:C_0402_small, symbol Device:C
- added D1: 1N5819WS, Diode_SMD:D_SOD-323, symbol Diode:1N5819WS
- added J3: FH12-30S-0.5SH_55_, lib:HIROSE_FH12-30S-0.5SH_55_, symbol FH12-30S-0.5SH_55_:FH12-30S-0.5SH_55_
- added L1: L, Inductor_SMD:L_1210_3225Metric, symbol Device:L
- added R11: 4.7, Resistor_SMD:R_0402_1005Metric, symbol Device:R
- added R5: 2, Resistor_SMD:R_0402_1005Metric, symbol Device:R
- added U1: TPS61042DRBR, lib:DRB8_1P75X1P5, symbol TPS61042:TPS61042DRBR
Connections:
- net  LED_A: now also C35.2, D1.1 (K), J3.30, U1.7 (OVP)
- net  LED_K: now also J3.28, J3.29, U1.1 (LED)
- net +2V8: now also C5.2, C6.1, J3.2, J3.27
- net D2_N: now also J3.11
- net D2_P: now also J3.12
- net LCM_ID: now also J3.1
- net PWM: now also J3.23
- net RESET: now also J3.25
- net TE: now also J3.24
- net TP_INT: now also J3.6
- net TP_RES: now also J3.3
- net TP_SCL: now also J3.4
- net TP_SDA: now also J3.5
- new net: R11.2, R5.1
- new net: R5.2, U1.2 (RS), U1.4 (FB)
- new net: D1.2 (A), L1.2, U1.8 (SW)
- new net +1V8: C4.1, J3.26
- new net +3V3: C9.2, L1.1, U1.3 (VIN)
- new net D3_N: J3.8
- new net D3_P: J3.9
- new net DC_LED_PWM: U1.5 (CTRL)
- new net DSI_CK_N: J3.14
- new net DSI_CK_P: J3.15
- new net DSI_D0_N: J3.20
- new net DSI_D0_P: J3.21
- new net DSI_D1_N: J3.17
- new net DSI_D1_P: J3.18
- new net GND: C35.1, C4.2, C5.1, C6.2, C7.2, C8.2, C9.1, J3.10, J3.13, J3.16, J3.19, J3.22, J3.7, J3.S1 (SHIELD), J3.S2 (SHIELD__1), R11.1, U1.6 (GND), U1.9 (EPAD)
- new net VDD_DDR: C7.1, C8.1
- no-connect marks 2 -> 0
Other:
- note added: "The traces use the **VDD_DDR** reference plane."
- note removed: "WRONG PART. SHOULD BE WITH PINS FACING FROM TOP TO BOTTOM"
