File: PCB/USB.kicad_sch (KiCad schematic)
At the start: 17 parts, among them J1 USB4510-03-1-A_REVA, J1101 USB4510-03-1-A_REVA, U1101 HSP051-4M10, U2 HSP051-4M10

Commit message: UPDATE
Connections:
- net USB_CC1: no longer J1.A5 (CC1)
- net USB_M_CC1: now also J1.A5 (CC1)
Changed lines of the file:
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@@
 		)
 	)
-	(global_label "USB_CC1"
+	(global_label "USB_M_CC1"
 		(shape input)
 		(at 88.9 118.11 180)
@@
 		)
 		(property "Intersheetrefs" "${INTERSHEET_REFS}"
-			(at 77.3877 118.11 0)
+			(at 74.9687 118.11 0)
 			(effects
 				(font

Commit message: PCB_UPDATE
Parts:
- added D7: LED_B, LED_SMD:LED_0402_1005Metric, symbol Device:LED
- added R7: ~, Resistor_SMD:R_0402_1005Metric, symbol Device:R
Connections:
- net GND: now also D7.1 (K)
- net VIN: now also R7.2
- new net: D7.2 (A), R7.1
Other:
- note added: "Need R calc"
