File: LCD_Adapter/LCD_Adapter_HAT/LCD_Adapter.kicad_pcb (KiCad board)
At the start: 4 copper layers, 100 x 70 mm, 68 parts, among them J2 FH12-30S-0.5SH_55_, J3 RPi_GPIO, J6 2-1734248-0, Q1 2N7002, Q2 2N7002, U1 TLV75801PDBV, U2 TLV75801PDBV, U3 TPS61042DRBR

Commit message: PCB_ADAPTER_UPDATE
Parts:
- removed J6: 2-1734248-0, lib:2-1734248-0
- removed R11: 0, Resistor_SMD:R_0603_1608Metric
- added C1: 0.47uF, Capacitor_SMD:C_0603_1608Metric, F.Cu at (200.3, 129.7)
- added C12: 0.47uF, Capacitor_SMD:C_0603_1608Metric, B.Cu at (81.1, 120.8)
- added C2: 4.7uF, Capacitor_SMD:C_0603_1608Metric, F.Cu at (201.8, 129.7)
- added C3: 0.47uF, Capacitor_SMD:C_0603_1608Metric, F.Cu at (198.1, 124.9)
- added C4: 0.47uF, Capacitor_SMD:C_0603_1608Metric, F.Cu at (207.2, 131.4)
- added C5: 0.47uF, Capacitor_SMD:C_0603_1608Metric, F.Cu at (203.4, 126.5)
- added C6: 4.7uF, Capacitor_SMD:C_0603_1608Metric, F.Cu at (204.9, 126.5)
- added C7: 1uF, Capacitor_SMD:C_0603_1608Metric, F.Cu at (213.4, 131.1)
- added C8: 4.7uF, Capacitor_SMD:C_0603_1608Metric, F.Cu at (213.4, 124.8)
- added D1: 1N5819WS, Diode_SMD:D_SOD-323, F.Cu at (216.5, 131.0)
- added J1: 2-84953-0, lib:TE_2-84953-0, B.Cu at (100.0, 114.0)
- added J4: Conn_02x20_Odd_Even, Connector_PinSocket_2.54mm:PinSocket_2x20_P2.54mm_Vertical_SMD, B.Cu at (114.0, 148.0)
- added L1: L, Inductor_SMD:L_1210_3225Metric, F.Cu at (218.3, 127.7)
- added R1: 330, Resistor_SMD:R_0603_1608Metric, B.Cu at (80.9, 143.6)
- added R12: 51k, Resistor_SMD:R_0603_1608Metric, F.Cu at (198.1, 131.9)
- added R13: 220k, Resistor_SMD:R_0603_1608Metric, F.Cu at (198.1, 130.5)
- added R14: 220k, Resistor_SMD:R_0603_1608Metric, F.Cu at (207.2, 125.7)
- added R15: 82k, Resistor_SMD:R_0603_1608Metric, F.Cu at (207.2, 124.3)
- added R16: 6.8, Resistor_SMD:R_0603_1608Metric, F.Cu at (211.4, 126.3)
- added R29: 330, Resistor_SMD:R_0603_1608Metric, B.Cu at (103.9, 107.6)
- added TP10: TestPoint, TestPoint:TestPoint_Pad_D1.0mm, F.Cu at (206.4, 121.1)
- added TP11: TestPoint, TestPoint:TestPoint_Pad_D1.0mm, F.Cu at (216.8, 121.1)
- added TP12: TestPoint, TestPoint:TestPoint_Pad_D1.0mm, F.Cu at (218.9, 121.1)
- added TP13: TestPoint, TestPoint:TestPoint_Pad_D1.0mm, F.Cu at (214.8, 121.1)
- added TP14: TestPoint, TestPoint:TestPoint_Pad_D1.0mm, F.Cu at (198.3, 121.2)
- added TP7: TestPoint, TestPoint:TestPoint_Pad_D1.0mm, F.Cu at (204.4, 121.1)
- added TP8: TestPoint, TestPoint:TestPoint_Pad_D1.0mm, F.Cu at (200.3, 121.2)
- added TP9: TestPoint, TestPoint:TestPoint_Pad_D1.0mm, F.Cu at (202.3, 121.1)
- added U1: TLV75801PDBV, Package_TO_SOT_SMD:SOT-23-5, F.Cu at (197.8, 127.7)
- added U2: TLV75801PDBV, Package_TO_SOT_SMD:SOT-23-5, F.Cu at (207.4, 128.5)
- added U3: TPS61042DRBR, lib:DRB8_1P75X1P5, F.Cu at (214.8, 127.8)
- added U4: PCA9306DCURG4, lib:SOP50P310X90-8N, B.Cu at (106.7, 123.5)
- added VD1: BAS70-06.215, lib:SOT23, B.Cu at (104.0, 105.0)
- C1, C10, C11, C13, C14, C15, C16, C2, C3, C4, C5, C6, C7, C8, C9, D1, J2, L1, Q1, Q2, R10, R12, R13, R14, R15, R16, R17, R18, R19, R2, R20, R21, R22, R23, R24, R25, R26, R27, R28, R4, R5, R6, R7, R8, R9, TP1, TP10, TP11, TP12, TP13, TP14, TP15, TP16, TP2, TP3, TP4, TP5, TP6, TP7, TP8, TP9, U1, U2, U3: moved to B.Cu
- R3: value 0 -> 330; moved to B.Cu
- moved J2 138.7 mm to (78.2, 114.0), turned to 90 degrees
- moved TP5 128.4 mm to (76.0, 145.6), turned to 180 degrees
- moved Q2 128.3 mm to (79.0, 146.2), turned to 180 degrees
- moved R7 127.2 mm to (81.7, 146.1), turned to 90 degrees
- moved C10 114.9 mm to (81.7, 107.3)
- moved C11 114.6 mm to (81.7, 108.8)
- moved R26 109.8 mm to (106.8, 130.1), turned to -90 degrees
- moved R27 109.6 mm to (105.2, 130.1), turned to -90 degrees
- moved Q1 108.7 mm to (85.5, 103.8), turned to 180 degrees
- moved R24 105.1 mm to (106.2, 115.8), turned to 90 degrees
- moved TP6 104.4 mm to (84.4, 101.0), turned to 180 degrees
- moved R6 104.1 mm to (88.3, 103.8), turned to 90 degrees
- moved R22 102.9 mm to (104.5, 127.8), turned to 180 degrees
- moved R25 102.6 mm to (107.7, 115.8), turned to 90 degrees
- moved R21 101.7 mm to (107.5, 127.8)
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Connections:
- C9 pad 1: +3V3 -> Net-(U4-EN)
- Q2 pad 1: TP_RES_STM_SIDE -> Net-(Q2-G)
- R7 pad 2: TP_RES_STM_SIDE -> Net-(Q2-G)
Routing:
- net /STM2LCD/D1_P: track 0.00 -> 28.7 mm
- net /STM2LCD/D1_N: track 0.00 -> 28.7 mm
- net /STM2LCD/CLK_N: track 0.00 -> 24.1 mm, vias 0 -> 2
- net /STM2LCD/CLK_P: track 0.00 -> 24.0 mm, vias 0 -> 2
- net /STM2LCD/D0_P: track 0.00 -> 23.8 mm
- net /STM2LCD/D0_N: track 0.00 -> 23.8 mm
- added copper zone on B.Cu, net GND
