File: LCD_Adapter/LCD_Adapter_HAT/LCD_Adapter.kicad_pcb (KiCad board)
At the start: 4 copper layers, 100 x 60 mm, 73 parts, among them J1 2-84953-0, J2 FH12-30S-0.5SH_55_, J3 RPi_GPIO, J4 Conn_02x20_Odd_Even, Q1 2N7002, Q2 2N7002, U1 TLV75801PDBV, U2 TLV75801PDBV, U3 TPS61042DRBR, U4 PCA9306DCURG4

Commit message: adapter update. maybe done
Parts:
- added R11: 4.7, Resistor_SMD:R_0603_1608Metric, B.Cu at (115.8, 136.0)
- R16: value 6.8 -> 2
Connections:
- R16 pad 1: GND -> Net-(R11-Pad2)
Routing:
- net /STM2LCD/D0_P: track 23.8 -> 28.6 mm
- net /STM2LCD/D0_N: track 23.8 -> 28.6 mm
- net  LED_A: track 88.9 -> 84.4 mm
- net GND: track 91.3 -> 88.7 mm, vias 76 -> 73
- net Net-(R11-Pad2): track 0.00 -> 1.61 mm
- net /STM2LCD/CLK_N: track 24.1 -> 25.6 mm
- net /STM2LCD/CLK_P: track 24.0 -> 25.5 mm
- net +2V8: track 139.8 -> 138.9 mm, vias 7 -> 6
