File: LCD_Adapter/LCD_Adapter_HAT/STM2LCD.kicad_sch (KiCad schematic)
At the start: 41 parts, among them J2 FH12-30S-0.5SH_55_, J3 RPi_GPIO, J6 2-1734248-0, Q1 2N7002, Q2 2N7002, U4 PCA9306DCURG4

Commit message: PCB_ADAPTER_UPDATE
Parts:
- removed J6: 2-1734248-0, CONN_2-1734248-0_TYCO, symbol 2-1734248-0:2-1734248-0
- removed R11: 0, Resistor_SMD:R_0603_1608Metric, symbol Device:R
- added C12: 0.47uF, Capacitor_SMD:C_0603_1608Metric, symbol Device:C
- added J1: 2-84953-0, lib:TE_2-84953-0, symbol 2-84953-0:2-84953-0
- added J4: Conn_02x20_Odd_Even, Connector_PinSocket_2.54mm:PinSocket_2x20_P2.54mm_Vertical_SMD, symbol Connector_Generic:Conn_02x20_Odd_Even
- added R1, R29: 330, Resistor_SMD:R_0603_1608Metric, symbol Device:R
- added VD1: BAS70-06.215, lib:SOT23, symbol BAS70-06.215:BAS70-06.215
- R3: value 0 -> 330; LCSC# (none) -> C23138
- U4: footprint PCA9306DCURG4:SOP50P310X90-8N -> lib:SOP50P310X90-8N
Connections:
- net +1V8: now also VD1.1 (K2)
- net +2V8: now also C12.2
- net +3V3: now also J1.14, J1.15; no longer C9.1
- net CLK_N: now also J1.5
- net CLK_P: now also J1.6
- net D0_N: now also J1.8
- net D0_P: now also J1.9
- net D1_N: now also J1.2
- net D1_P: now also J1.3
- net GND: now also C12.1, J1.1, J1.10, J1.13, J1.16, J1.4, J1.7, J1.S1 (SHIELD), J1.S2 (SHIELD)
- net TP_INT: now also R29.2, VD1.3 (A)
- net TP_RES_STM_SIDE: now also R1.1; no longer Q2.1 (G), R7.2
- net at R25.1: now also J1.11
- net at R3.1: now also J1.20
- net at R5.1: now also J1.19
- net at R24.1: now also J1.12
- net at R4.1: now also J1.18
- net at R23.1, U4.7 (VREF2), U4.8 (EN): now also C9.1
- new net: Q2.1 (G), R1.2, R7.2
- new net: J1.17, R29.1
- no-connect marks 0 -> 1
Other:
- moved on the sheet: C9, Q1, Q2, R6, R7, R8, R9, TP6
