File: LCD_Adapter/LCD_Adapter_HAT/STM2LCD.kicad_sch (KiCad schematic)
At the start: 45 parts, among them J1 2-84953-0, J2 FH12-30S-0.5SH_55_, J3 RPi_GPIO, J4 Conn_02x20_Odd_Even, Q1 2N7002, Q2 2N7002, U4 PCA9306DCURG4

Commit message: adapter update. maybe done
Parts:
- R6: now left out of the parts list
- VD1: LCSC# (none) -> C8651
Connections:
- no-connect marks 1 -> 77
