File: LCD_Adapter/LCD_Adapter_HAT/PWM.kicad_sch (KiCad schematic)
At the start: 29 parts, among them U1 TLV75801PDBV, U2 TLV75801PDBV, U3 TPS61042DRBR

Commit message: adapter update. maybe done
Parts:
- R11: value 6.8 -> 4.7; LCSC# (none) -> C23164
- R16: value 6.8 -> 2; LCSC# (none) -> C22977
Connections:
- net GND: now also R11.1
- net at R16.1: now also R11.2
Changed lines of the file:
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@@
 	(wire
 		(pts
+			(xy 124.46 162.56) (xy 124.46 163.83)
+		)
+		(stroke
+			(width 0)
+			(type default)
+		)
+	)
+	(wire
+		(pts
 			(xy 142.24 35.56) (xy 142.24 36.83)
 		)
@@
 	(wire
 		(pts
+			(xy 124.46 171.45) (xy 124.46 172.72)
+		)
+		(stroke
+			(width 0)
+			(type default)
+		)
+	)
+	(wire
+		(pts
 			(xy 80.01 135.89) (xy 80.01 125.73)
 		)
@@
 			)
 		)
-		(property "Value" "6.8"
+		(property "Value" "2"
 			(at 128.27 160.528 0)
 			(effects
@@
 			)
 		)
+		(property "LCSC#" "C22977"
+			(at 124.46 158.75 0)
+			(effects
+				(font
+					(size 1.27 1.27)
+				)
+				(hide yes)
+			)
+		)
 		(pin "1"
 		)
@@
 			)
 		)
-		(property "Value" "6.8"
+		(property "Value" "4.7"
 			(at 128.27 169.418 0)
 			(effects
@@
 			(at 124.46 167.64 0)
 			(effects
+				(font
+					(size 1.27 1.27)
+				)
+				(hide yes)
+			)
+		)
+		(property "LCSC#" "C23164"
+			(at 124.46 167.64 0)
+			(effects
