File: MAIN_PCB/FLASH_SD.kicad_sch (KiCad schematic)
At the start: 13 parts, among them J501 MEM2090-00-145-00-A_REVA, U501 HSP051-4M10, U502 HSP051-4M10

Commit message: UPDATE
Other:
- company: (none) -> COMPANY_NAME
Changed lines of the file:
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@@
 	(paper "A3")
 	(title_block
+		(company "COMPANY_NAME")
 		(comment 1 "Author: Mykola Grodskyi")
+		(comment 2 "Copyright © 2025 Mykola Grodskyi.")
+		(comment 3 "Licensed under CERN-OHL-S v2 (see LICENSE for details)")
+		(comment 4 "PROVIDED \"AS IS\" WITHOUT WARRANTY OF ANY KIND")
+		(comment 5 "Source: github.com/")
 	)
 	(text "CHECKED 2.0 MG\n"

Commit message: UPDATE
Other:
- company: COMPANY_NAME -> DECKTRIX-LAB
- title: (none) -> DECKTRIX
Changed lines of the file:
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@@
 	(paper "A3")
 	(title_block
-		(company "COMPANY_NAME")
+		(title "DECKTRIX")
+		(company "DECKTRIX-LAB")
 		(comment 1 "Author: Mykola Grodskyi")
 		(comment 2 "Copyright © 2025 Mykola Grodskyi.")
 		(comment 3 "Licensed under CERN-OHL-S v2 (see LICENSE for details)")
 		(comment 4 "PROVIDED \"AS IS\" WITHOUT WARRANTY OF ANY KIND")
-		(comment 5 "Source: github.com/")
+		(comment 5 "Source: https://github.com/Decktrix-Lab/decktrix")
 	)
 	(text "CHECKED 2.0 MG\n"

Commit message: UPDATE
Parts:
- renumbered R8 to R504
Changed lines of the file:
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@@
 		(dnp no)
 		(fields_autoplaced yes)
-		(property "Reference" "R8"
+		(property "Reference" "R504"
 			(at 304.8 120.6499 0)
 			(effects
@@
 			(project "MPU_MOD"
 				(path "/65890f61-d586-475b-928a-b635a5e4e59e/ec317a3c-922b-4ac6-af1a-f2cdb70bc7c5"
-					(reference "R8")
+					(reference "R504")
 					(unit 1)
 				)

Commit message: UPDATE
Other:
- note removed: "CHECKED 2.0 MG"
Changed lines of the file:
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@@
 		(comment 5 "Source: https://github.com/Decktrix-Lab/decktrix")
-	)
-	(text "CHECKED 2.0 MG\n"
-		(exclude_from_sim no)
-		(at 164.084 123.19 0)
-		(effects
-			(font
-				(size 12.7 12.7)
-				(color 97 255 51 1)
-			)
-		)
 	)
 	(junction
