File: MAIN_PCB/HS_intrf.kicad_sch (KiCad schematic)
At the start: 2 parts, among them U4 STM32MP157FABx

Commit message: UPDATE
Connections:
- no-connect marks 0 -> 1
Other:
- note added: "CHECKED 2.0 MG"
Changed lines of the file:
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@@
 		(comment 5 "Source: github.com/")
+	)
+	(text "CHECKED 2.0 MG\n"
+		(exclude_from_sim no)
+		(at 101.346 44.45 0)
+		(effects
+			(font
+				(size 12.7 12.7)
+				(color 97 255 51 1)
+			)
+		)
 	)
 	(text_box "VSS_USBHS\n"
@@
 			(justify left top)
 		)
+	)
+	(no_connect
+		(at 83.82 66.04)
 	)
 	(wire
@@
 		(on_board yes)
 		(dnp no)
-		(fields_autoplaced yes)
 		(property "Reference" "U4"
 			(at -68.58 240.03 0)
@@
 		)
 		(property "Value" "STM32MP157FABx"
-			(at 63.5 160.02 90)
-			(effects
-				(font
+			(at 106.68 83.058 0)
+			(effects
+				(font

Commit message: UPDATE
Other:
- company: COMPANY_NAME -> DECKTRIX-LAB
- title: (none) -> DECKTRIX
Changed lines of the file:
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@@
 	(paper "A3")
 	(title_block
-		(company "COMPANY_NAME")
+		(title "DECKTRIX")
+		(company "DECKTRIX-LAB")
 		(comment 1 "Author: Mykola Grodskyi")
 		(comment 2 "Copyright © 2025 Mykola Grodskyi.")
 		(comment 3 "Licensed under CERN-OHL-S v2 (see LICENSE for details)")
 		(comment 4 "PROVIDED \"AS IS\" WITHOUT WARRANTY OF ANY KIND")
-		(comment 5 "Source: github.com/")
+		(comment 5 "Source: https://github.com/Decktrix-Lab/decktrix")
 	)
 	(text "CHECKED 2.0 MG\n"

Commit message: UPDATE
Parts:
- U301: renamed from U4; Mouser P/N (none) -> 511-STM32MP157FAB1; REC P/N (none) -> STM32MP157FAB1
Changed lines of the file:
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@@
 		(on_board yes)
 		(dnp no)
-		(property "Reference" "U4"
+		(property "Reference" "U301"
 			(at -68.58 240.03 0)
 			(effects
@@
 		)
 		(property "VENDOR" ""
+			(at 87.63 82.55 0)
+			(effects
+				(font
+					(size 1.27 1.27)
+				)
+				(hide yes)
+			)
+		)
+		(property "Mouser P/N" "511-STM32MP157FAB1"
+			(at 87.63 82.55 0)
+			(effects
+				(font
+					(size 1.27 1.27)
+				)
+				(hide yes)
+			)
+		)
+		(property "REC P/N" "STM32MP157FAB1"
 			(at 87.63 82.55 0)
 			(effects
@@
 			(project "MPU_MOD"
 				(path "/65890f61-d586-475b-928a-b635a5e4e59e/9899e005-10ba-4bf4-b936-8d0d8a1813b9"
-					(reference "U4")
+					(reference "U301")
 					(unit 6)
 				)

Commit message: UPDATE
Other:
- note removed: "CHECKED 2.0 MG"
Changed lines of the file:
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@@
 		(comment 5 "Source: https://github.com/Decktrix-Lab/decktrix")
-	)
-	(text "CHECKED 2.0 MG\n"
-		(exclude_from_sim no)
-		(at 101.346 44.45 0)
-		(effects
-			(font
-				(size 12.7 12.7)
-				(color 97 255 51 1)
-			)
-		)
 	)
 	(text_box "VSS_USBHS\n"
