File: MAIN_PCB/IO_Perph_Conn.kicad_sch (KiCad schematic)
At the start: 23 parts, among them J3 M40-3100645R, U3 HSP051-4M10, U4 STM32MP157FABx, U5 HSP051-4M10, Y601 NX2012SA-32.768K

Commit message: UPDATE
Other:
- company: (none) -> COMPANY_NAME
Changed lines of the file:
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@@
 	(paper "A3")
 	(title_block
+		(company "COMPANY_NAME")
 		(comment 1 "Author: Mykola Grodskyi")
+		(comment 2 "Copyright © 2025 Mykola Grodskyi.")
+		(comment 3 "Licensed under CERN-OHL-S v2 (see LICENSE for details)")
+		(comment 4 "PROVIDED \"AS IS\" WITHOUT WARRANTY OF ANY KIND")
+		(comment 5 "Source: github.com/")
 	)
 	(text "Need R calc\n"

Commit message: UPDATE
Other:
- company: COMPANY_NAME -> DECKTRIX-LAB
- title: (none) -> DECKTRIX
Changed lines of the file:
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@@
 	(paper "A3")
 	(title_block
-		(company "COMPANY_NAME")
+		(title "DECKTRIX")
+		(company "DECKTRIX-LAB")
 		(comment 1 "Author: Mykola Grodskyi")
 		(comment 2 "Copyright © 2025 Mykola Grodskyi.")
 		(comment 3 "Licensed under CERN-OHL-S v2 (see LICENSE for details)")
 		(comment 4 "PROVIDED \"AS IS\" WITHOUT WARRANTY OF ANY KIND")
-		(comment 5 "Source: github.com/")
+		(comment 5 "Source: https://github.com/Decktrix-Lab/decktrix")
 	)
 	(text "Need R calc\n"

Commit message: mod_before_brake
Connections:
- no-connect marks 23 -> 24
Other:
- note added: "CHECKED 2.0 MG"

Commit message: UPDATE
Parts:
- J601: renamed from J3; Mouser P/N (none) -> 855-M40-3100645R; REC P/N (none) -> M40-3100645R
- R601, R602: value ~ -> 33; LCSC Part # (none) -> C138002
- TP601, TP602, TP603, TP604, TP605: LCSC Part # (none) -> DNI; Mouser P/N (none) -> DNI; REC P/N (none) -> DNI
- U301: renamed from U4; Mouser P/N (none) -> 511-STM32MP157FAB1; REC P/N (none) -> STM32MP157FAB1
- Y601: REC P/N (none) -> NX2012SA-32.768K
- renumbered D2 to D603, D4 to D604, D5 to D605, U3 to U601, U5 to U602
Other:
- note removed: "Need R calc"

Commit message: UPDATE
Other:
- note removed: "CHECKED 2.0 MG"
Changed lines of the file:
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@@
 		(comment 5 "Source: https://github.com/Decktrix-Lab/decktrix")
-	)
-	(text "CHECKED 2.0 MG\n"
-		(exclude_from_sim no)
-		(at 178.816 28.194 0)
-		(effects
-			(font
-				(size 12.7 12.7)
-				(color 97 255 51 1)
-			)
-		)
 	)
 	(junction
