File: MAIN_PCB/LCD.kicad_sch (KiCad schematic)
At the start: 30 parts, among them J1001 FH12-30S-0.5SH_55_, Q1 DMG1012TQ-7, Q2 DMG1012TQ-7, Q3 DMG1012TQ-7, U1001 TPS61042DRBR

Commit message: UPDATE
Other:
- company: (none) -> COMPANY_NAME
Changed lines of the file:
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@@
 	(generator "eeschema")
 	(generator_version "9.0")
-	(paper "A4")
+	(paper "A3")
+	(title_block
+		(company "COMPANY_NAME")
+		(comment 1 "Author: Mykola Grodskyi")
+		(comment 2 "Copyright © 2025 Mykola Grodskyi.")
+		(comment 3 "Licensed under CERN-OHL-S v2 (see LICENSE for details)")
+		(comment 4 "PROVIDED \"AS IS\" WITHOUT WARRANTY OF ANY KIND")
+		(comment 5 "Source: github.com/")
+	)
 	(text "NEED REVIEW"
 		(exclude_from_sim no)

Commit message: UPDATE
Other:
- note added: "CHECKED 2.0 MG"
- note removed: "NEED REVIEW"
- company: COMPANY_NAME -> DECKTRIX-LAB
- title: (none) -> DECKTRIX
Changed lines of the file:
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@@
 	(paper "A3")
 	(title_block
-		(company "COMPANY_NAME")
+		(title "DECKTRIX")
+		(company "DECKTRIX-LAB")
 		(comment 1 "Author: Mykola Grodskyi")
 		(comment 2 "Copyright © 2025 Mykola Grodskyi.")
 		(comment 3 "Licensed under CERN-OHL-S v2 (see LICENSE for details)")
 		(comment 4 "PROVIDED \"AS IS\" WITHOUT WARRANTY OF ANY KIND")
-		(comment 5 "Source: github.com/")
-	)
-	(text "NEED REVIEW"
-		(exclude_from_sim no)
-		(at 88.646 99.822 0)
-		(effects
-			(font
-				(size 2.54 2.54)
-				(color 255 41 58 1)
-			)
-		)
+		(comment 5 "Source: https://github.com/Decktrix-Lab/decktrix")
 	)
 	(text "The traces use the **VDD_DDR** reference plane."
@@
 			)
 		)
+	)
+	(text "CHECKED 2.0 MG\n"
+		(exclude_from_sim no)
+		(at 178.562 235.712 0)
+		(effects
+			(font
+				(size 12.7 12.7)
+				(color 97 255 51 1)
+			)
+		)

Commit message: update
Parts:
- added C1008: 100nF, lib:C_0402_small, symbol Device:C
Connections:
- net GND: now also C1008.2
- net VDD_DDR: now also C1008.1

Commit message: UPDATE
Parts:
- C1003, C1005: Mouser P/N (none) -> 81-GRM155R61E104KA7J; REC P/N (none) -> GRM155R61E104KA87J
- C1004: Mouser P/N (none) -> 81-GRM155R61E105KA2D
- C1006: renamed from C1008; Mouser P/N (none) -> 81-GRM155R61E104KA7J; REC P/N (none) -> GRM155R61E104KA87J
- C1007: renamed from C1006; Mouser P/N (none) -> 81-GRM155R61E105KA2D
- C1008: renamed from C1007; Mouser P/N (none) -> 81-GRM155R61E105KA2D
- Q1001: renamed from Q1; LCSC Part # (none) -> C531154
- Q1002: renamed from Q2; LCSC Part # (none) -> C531154
- Q1003: renamed from Q3; LCSC Part # (none) -> C531154
- TP1001, TP1002, TP1003, TP1004, TP1005, TP1006: LCSC Part # (none) -> DNI; Mouser P/N (none) -> DNI; REC P/N (none) -> DNI
- U1001: REC P/N (none) -> TPS61042DRBR

Commit message: UPDATE
Other:
- note removed: "CHECKED 2.0 MG"
Changed lines of the file:
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@@
-		)
-	)
-	(text "CHECKED 2.0 MG\n"
-		(exclude_from_sim no)
-		(at 178.562 235.712 0)
-		(effects
-			(font
-				(size 12.7 12.7)
-				(color 97 255 51 1)
-			)
 		)
 	)
