File: MAIN_PCB/MPU_PWR.kicad_sch (KiCad schematic)
At the start: 47 parts, among them U4 STM32MP157FABx

Commit message: UPDATE
Other:
- company: (none) -> COMPANY_NAME
Changed lines of the file:
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@@
 	(paper "A3")
 	(title_block
+		(company "COMPANY_NAME")
 		(comment 1 "Author: Mykola Grodskyi")
+		(comment 2 "Copyright © 2025 Mykola Grodskyi.")
+		(comment 3 "Licensed under CERN-OHL-S v2 (see LICENSE for details)")
+		(comment 4 "PROVIDED \"AS IS\" WITHOUT WARRANTY OF ANY KIND")
+		(comment 5 "Source: github.com/")
 	)
 	(text "CHECKED 2.0 MG\n"

Commit message: UPDATE
Other:
- company: COMPANY_NAME -> DECKTRIX-LAB
- title: (none) -> DECKTRIX
Changed lines of the file:
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@@
 	(paper "A3")
 	(title_block
-		(company "COMPANY_NAME")
+		(title "DECKTRIX")
+		(company "DECKTRIX-LAB")
 		(comment 1 "Author: Mykola Grodskyi")
 		(comment 2 "Copyright © 2025 Mykola Grodskyi.")
 		(comment 3 "Licensed under CERN-OHL-S v2 (see LICENSE for details)")
 		(comment 4 "PROVIDED \"AS IS\" WITHOUT WARRANTY OF ANY KIND")
-		(comment 5 "Source: github.com/")
+		(comment 5 "Source: https://github.com/Decktrix-Lab/decktrix")
 	)
 	(text "CHECKED 2.0 MG\n"

Commit message: UPDATE
Parts:
- C338: Mouser P/N (none) -> 628-CPH3225A; REC P/N (none) -> CPH3225A
- U301: renamed from U4; Mouser P/N (none) -> 511-STM32MP157FAB1; REC P/N (none) -> STM32MP157FAB1
Changed lines of the file:
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@@
 		(dnp no)
 		(fields_autoplaced yes)
-		(property "Reference" "U4"
+		(property "Reference" "U301"
 			(at 43.18 284.48 0)
 			(effects
@@
 			)
 		)
+		(property "Mouser P/N" "511-STM32MP157FAB1"
+			(at 199.39 127 0)
+			(effects
+				(font
+					(size 1.27 1.27)
+				)
+				(hide yes)
+			)
+		)
+		(property "REC P/N" "STM32MP157FAB1"
+			(at 199.39 127 0)
+			(effects
+				(font
+					(size 1.27 1.27)
+				)
+				(hide yes)
+			)
+		)
 		(pin "T9"
 		)
@@
 				)
 				(path "/65890f61-d586-475b-928a-b635a5e4e59e/f922126e-a4bd-4f88-a222-a0ba90de18ce"
-					(reference "U4")
+					(reference "U301")
 					(unit 1)
 				)
@@
 			(at 139.7 26.67 90)
 			(effects
+				(font
+					(size 1.27 1.27)
+				)
+				(hide yes)
+			)
+		)
+		(property "Mouser P/N" "628-CPH3225A"
+			(at 139.7 26.67 90)
+			(effects
+				(font
+					(size 1.27 1.27)
+				)
+				(hide yes)
+			)
+		)
+		(property "REC P/N" "CPH3225A"
+			(at 139.7 26.67 90)
+			(effects

Commit message: FabFile_ready
Parts:
- L301: value 1uH -> 4.7uH
Changed lines of the file:
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@@
 			)
 		)
-		(property "Value" "1uH"
+		(property "Value" "4.7uH"
 			(at 105.156 110.236 90)
 			(effects

Commit message: UPDATE
Other:
- note removed: "CHECKED 2.0 MG"
Changed lines of the file:
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@@
 		(comment 5 "Source: https://github.com/Decktrix-Lab/decktrix")
-	)
-	(text "CHECKED 2.0 MG\n"
-		(exclude_from_sim no)
-		(at 145.288 77.216 0)
-		(effects
-			(font
-				(size 12.7 12.7)
-				(color 97 255 51 1)
-			)
-		)
 	)
 	(junction
