File: MAIN_PCB/PWR.kicad_sch (KiCad schematic)
At the start: 47 parts, among them Q201 DMG1013T-7, U201 TPS62840DLCR, U202 STPMIC1APQR

Commit message: UPDATE
Other:
- company: (none) -> COMPANY_NAME
Changed lines of the file:
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@@
 	(paper "A3")
 	(title_block
+		(company "COMPANY_NAME")
 		(comment 1 "Author: Mykola Grodskyi")
+		(comment 2 "Copyright © 2025 Mykola Grodskyi.")
+		(comment 3 "Licensed under CERN-OHL-S v2 (see LICENSE for details)")
+		(comment 4 "PROVIDED \"AS IS\" WITHOUT WARRANTY OF ANY KIND")
+		(comment 5 "Source: github.com/")
 	)
 	(text "Caution: VDD3V3_USBHS must not be present unless VDDA1V8_REG is present, otherwise permanent\nSTM32MP15x lines damage can occur. It must be ensured by PMIC ranking order or with\nexternal component in case of discrete component power-supply implementation."

Commit message: UPDATE
Other:
- company: COMPANY_NAME -> DECKTRIX-LAB
- title: (none) -> DECKTRIX
Changed lines of the file:
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@@
 	(paper "A3")
 	(title_block
-		(company "COMPANY_NAME")
+		(title "DECKTRIX")
+		(company "DECKTRIX-LAB")
 		(comment 1 "Author: Mykola Grodskyi")
 		(comment 2 "Copyright © 2025 Mykola Grodskyi.")
 		(comment 3 "Licensed under CERN-OHL-S v2 (see LICENSE for details)")
 		(comment 4 "PROVIDED \"AS IS\" WITHOUT WARRANTY OF ANY KIND")
-		(comment 5 "Source: github.com/")
+		(comment 5 "Source: https://github.com/Decktrix-Lab/decktrix")
 	)
 	(text "Caution: VDD3V3_USBHS must not be present unless VDDA1V8_REG is present, otherwise permanent\nSTM32MP15x lines damage can occur. It must be ensured by PMIC ranking order or with\nexternal component in case of discrete component power-supply implementation."

Commit message: UPDATE
Parts:
- L201: LCSC Part # (none) -> C337893
- Q201: LCSC Part # (none) -> C96676
- S201: renamed from S2; LCSC Part # (none) -> C963349
- TP201, TP202, TP203, TP204, TP205, TP206, TP207, TP208, TP209, TP210, TP211: LCSC Part # (none) -> DNI; Mouser P/N (none) -> DNI; REC P/N (none) -> DNI
- U201: LCSC Part # (none) -> C2071859
- renumbered D3 to D201

Commit message: UPDATE
Other:
- note removed: "CHECKED 2.0 MG"
