File: MAIN_PCB/RCC_BOOT_RST_DEBUG.kicad_sch (KiCad schematic)
At the start: 31 parts, among them J701 FTSH-107-01-L-DV-K-A, U4 STM32MP157FABx, U702 HSP051-4M10, U703 HSP051-4M10, Y701 ECS-2520MVQ-240

Commit message: UPDATE
Other:
- company: (none) -> COMPANY_NAME
Changed lines of the file:
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@@
 	(paper "A3")
 	(title_block
+		(company "COMPANY_NAME")
 		(comment 1 "Author: Mykola Grodskyi")
+		(comment 2 "Copyright © 2025 Mykola Grodskyi.")
+		(comment 3 "Licensed under CERN-OHL-S v2 (see LICENSE for details)")
+		(comment 4 "PROVIDED \"AS IS\" WITHOUT WARRANTY OF ANY KIND")
+		(comment 5 "Source: github.com/")
 	)
 	(text "CHECKED 2.0 MG\n"

Commit message: UPDATE
Other:
- company: COMPANY_NAME -> DECKTRIX-LAB
- title: (none) -> DECKTRIX
Changed lines of the file:
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@@
 	(paper "A3")
 	(title_block
-		(company "COMPANY_NAME")
+		(title "DECKTRIX")
+		(company "DECKTRIX-LAB")
 		(comment 1 "Author: Mykola Grodskyi")
 		(comment 2 "Copyright © 2025 Mykola Grodskyi.")
 		(comment 3 "Licensed under CERN-OHL-S v2 (see LICENSE for details)")
 		(comment 4 "PROVIDED \"AS IS\" WITHOUT WARRANTY OF ANY KIND")
-		(comment 5 "Source: github.com/")
+		(comment 5 "Source: https://github.com/Decktrix-Lab/decktrix")
 	)
 	(text "CHECKED 2.0 MG\n"

Commit message: UPDATE
Parts:
- J701: LCSC Part # (none) -> C5563894
- S701: renamed from S1; LCSC Part # (none) -> C963349
- TP701, TP702, TP703, TP704, TP705, TP706, TP707: LCSC Part # (none) -> DNI; Mouser P/N (none) -> DNI; REC P/N (none) -> DNI
- U301: renamed from U4; Mouser P/N (none) -> 511-STM32MP157FAB1; REC P/N (none) -> STM32MP157FAB1
- renumbered D6 to D701, U702 to U701, U703 to U702

Commit message: UPDATE
Other:
- note removed: "CHECKED 2.0 MG"
Changed lines of the file:
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@@
 		(comment 5 "Source: https://github.com/Decktrix-Lab/decktrix")
 	)
-	(text "CHECKED 2.0 MG\n"
-		(exclude_from_sim no)
-		(at 138.684 32.004 0)
-		(effects
-			(font
-				(size 12.7 12.7)
-				(color 97 255 51 1)
-			)
-		)
-	)
 	(junction
 		(at 297.18 52.07)
@@
 		(dnp no)
 		(property "Reference" "U301"
-			(at 35.56 270.51 0)
+			(at 196.85 100.33 0)
 			(effects
 				(font
