File: MAIN_PCB/USB.kicad_sch (KiCad schematic)
At the start: 19 parts, among them J1 USB4510-03-1-A_REVA, J1101 USB4510-03-1-A_REVA, U1101 HSP051-4M10, U2 HSP051-4M10

Commit message: UPDATE
Other:
- company: (none) -> COMPANY_NAME
Changed lines of the file:
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@@
 	(generator_version "9.0")
 	(paper "A3")
+	(title_block
+		(company "COMPANY_NAME")
+		(comment 1 "Author: Mykola Grodskyi")
+		(comment 2 "Copyright © 2025 Mykola Grodskyi.")
+		(comment 3 "Licensed under CERN-OHL-S v2 (see LICENSE for details)")
+		(comment 4 "PROVIDED \"AS IS\" WITHOUT WARRANTY OF ANY KIND")
+		(comment 5 "Source: github.com/")
+	)
 	(text "Need R calc\n"
 		(exclude_from_sim no)

Commit message: UPDATE
Other:
- note added: "CHECKED 2.0 MG"
- company: COMPANY_NAME -> DECKTRIX-LAB
- title: (none) -> DECKTRIX
Changed lines of the file:
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@@
 	(paper "A3")
 	(title_block
-		(company "COMPANY_NAME")
+		(title "DECKTRIX")
+		(company "DECKTRIX-LAB")
 		(comment 1 "Author: Mykola Grodskyi")
 		(comment 2 "Copyright © 2025 Mykola Grodskyi.")
 		(comment 3 "Licensed under CERN-OHL-S v2 (see LICENSE for details)")
 		(comment 4 "PROVIDED \"AS IS\" WITHOUT WARRANTY OF ANY KIND")
-		(comment 5 "Source: github.com/")
+		(comment 5 "Source: https://github.com/Decktrix-Lab/decktrix")
+	)
+	(text "CHECKED 2.0 MG\n"
+		(exclude_from_sim no)
+		(at 178.308 54.864 0)
+		(effects
+			(font
+				(size 12.7 12.7)
+				(color 97 255 51 1)
+			)
+		)
 	)
 	(text "Need R calc\n"

Commit message: UPDATE
Parts:
- R1101: renamed from R5; LCSC Part # (none) -> C114756
- R1102: renamed from R4; LCSC Part # (none) -> C114756
- R1103: renamed from R7; value ~ -> 240; LCSC Part # (none) -> C25094
- TP1101: LCSC Part # (none) -> DNI; Mouser P/N (none) -> DNI; REC P/N (none) -> DNI
- renumbered C7 to C1101, C8 to C1102, C9 to C1103, C1101 to C1104, C1102 to C1105, C1103 to C1106, D1 to D1101, D7 to D1102, D1101 to D1103, J1 to J1101, J1101 to J1102, R1101 to R1104, R1102 to R1105, U2 to U1101, U1101 to U1102
Other:
- note removed: "Need R calc"

Commit message: UPDATE
Other:
- note removed: "CHECKED 2.0 MG"
Changed lines of the file:
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@@
 		(comment 5 "Source: https://github.com/Decktrix-Lab/decktrix")
-	)
-	(text "CHECKED 2.0 MG\n"
-		(exclude_from_sim no)
-		(at 178.308 54.864 0)
-		(effects
-			(font
-				(size 12.7 12.7)
-				(color 97 255 51 1)
-			)
-		)
 	)
 	(junction
