File: MAIN_PCB/WIFI.kicad_sch (KiCad schematic)
At the start: 25 parts, among them U1 SIT1533AI-H4-DCC-32.768E, U901 MAYA-W166-00B

Commit message: UPDATE
Other:
- company: (none) -> COMPANY_NAME
Changed lines of the file:
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@@
 	(generator "eeschema")
 	(generator_version "9.0")
-	(paper "A4")
+	(paper "A3")
+	(title_block
+		(company "COMPANY_NAME")
+		(comment 1 "Author: Mykola Grodskyi")
+		(comment 2 "Copyright © 2025 Mykola Grodskyi.")
+		(comment 3 "Licensed under CERN-OHL-S v2 (see LICENSE for details)")
+		(comment 4 "PROVIDED \"AS IS\" WITHOUT WARRANTY OF ANY KIND")
+		(comment 5 "Source: github.com/")
+	)
 	(text "Conf settings during boot. internal pull-up exist. \nDon't interfere with it through UART or a pull-down on the input."
 		(exclude_from_sim no)

Commit message: UPDATE
Other:
- moved on the sheet: C1, C2, C3, C4, C5, C6, C901, C902, R1, R2, R3, R6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

Commit message: UPDATE
Other:
- note added: "CHECKED 2.0 MG"
- company: COMPANY_NAME -> DECKTRIX-LAB
- title: (none) -> DECKTRIX
Changed lines of the file:
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@@
 	(paper "A3")
 	(title_block
-		(company "COMPANY_NAME")
+		(title "DECKTRIX")
+		(company "DECKTRIX-LAB")
 		(comment 1 "Author: Mykola Grodskyi")
 		(comment 2 "Copyright © 2025 Mykola Grodskyi.")
 		(comment 3 "Licensed under CERN-OHL-S v2 (see LICENSE for details)")
 		(comment 4 "PROVIDED \"AS IS\" WITHOUT WARRANTY OF ANY KIND")
-		(comment 5 "Source: github.com/")
+		(comment 5 "Source: https://github.com/Decktrix-Lab/decktrix")
+	)
+	(text "CHECKED 2.0 MG\n"
+		(exclude_from_sim no)
+		(at 95.25 34.544 0)
+		(effects
+			(font
+				(size 12.7 12.7)
+				(color 97 255 51 1)
+			)
+		)
 	)
 	(text "Conf settings during boot. internal pull-up exist. \nDon't interfere with it through UART or a pull-down on the input."

Commit message: UPDATE
Parts:
- R902: renamed from R6; LCSC Part # (none) -> C114756
- R907, R908, R909, R910, R911, R912: LCSC Part # (none) -> C138002
- R914: renamed from R3; LCSC Part # (none) -> C138002
- U901: Mouser P/N (none) -> 377-MAYA-W166-00B; REC P/N (none) -> MAYA-W166-00B
- U902: renamed from U1; Mouser P/N (none) -> 788-1533AIH4DCC32.76; REC P/N (none) -> SiT1533AI-H4-DCC-32.768E
- renumbered C1 to C901, C5 to C902, C4 to C903, C901 to C904, C902 to C905, C6 to C906, C3 to C907, C2 to C908, R1 to R913, R2 to R915

Commit message: UPDATE
Other:
- note removed: "CHECKED 2.0 MG"
Changed lines of the file:
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@@
 		(comment 5 "Source: https://github.com/Decktrix-Lab/decktrix")
-	)
-	(text "CHECKED 2.0 MG\n"
-		(exclude_from_sim no)
-		(at 95.25 34.544 0)
-		(effects
-			(font
-				(size 12.7 12.7)
-				(color 97 255 51 1)
-			)
-		)
 	)
 	(text "Conf settings during boot. internal pull-up exist. \nDon't interfere with it through UART or a pull-down on the input."
