File: multimeter/Analog_Input.kicad_sch (KiCad schematic)
At the start: 18 parts, among them J201 Conn_01x01_Socket, J202 Conn_01x01_Socket, Q201 Si2301, Q202 Si2301, U201 TS5A3157DBVR, U202 ADS1115IDGS

Commit message: Update
Parts:
- removed U202: ADS1115IDGS, Package_SO:TSSOP-10_3x3mm_P0.5mm, symbol Analog_ADC:ADS1115IDGS
- added C201, C203: 100nF, symbol Device:C
- added C202: 1uF, symbol Device:C
- added C204: 10nF, symbol Device:C
- added R212, R213: 10k, symbol Device:R
- added R214: 100, symbol Device:R
- added U203: MCP6001-OT, Package_TO_SOT_SMD:SOT-23-5, symbol Amplifier_Operational:MCP6001-OT
Connections:
- net +3V3: now also R212.2
- net GND: now also C201.2, C202.2, R213.1
- net at D203.3 (K1A2), R210.2: now also C203.1
- net DMM_N_ADC: now reaches D203.6 (K3A4), R211.2
- net DMM_N_ADC: now also C203.2
- net at R202.2, R203.1, U201.1 (NO): now also C204.1
- net at J201.1 (Pin_1), R203.2, R211.1: now also C202.1, C204.2, R214.1
- new net: R214.2, U203.1, U203.4 (-)
- new net: C201.1, R212.1, R213.2, U203.3 (+)
Other:
- note added: "OP amp"
- note added: "REPLACE"
- moved on the sheet: D203A, D203B, R211

Commit message: UPDATE
Parts:
- removed D203: BAV199DW, Package_TO_SOT_SMD:SOT-363_SC-70-6, symbol Diode:BAV199DW
- added R215: 100, symbol Device:R
- added U302: OPA4322AIPWR, Package_SO:TSSOP-14_4.4x5mm_P0.65mm, symbol New_Library:OPA4322
- R210, R211: value 2K2 -> 100
Connections:
- net DMM_N_ADC: now also C202.1, R214.1
- net DMM_P_ADC: now also R215.2
- net at C203.1, R210.2: now also U302.12 (+)
- net at C204.2, J201.1 (Pin_1), R203.2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: no longer C202.1, R214.1
- new net: R215.1, U302.13 (-), U302.14
Other:
- note removed: "OP amp"
- moved on the sheet: C201, C202, C204, J201, J202, R203, R212, R213, R214, U201, U203
